File: design/RS232.sch (KiCad schematic (older format))
At the start: 0 parts

Commit message: Adding RS-232 Ports
Parts:
- added C? (x5): 0u1F, Capacitors_SMD:C_0603, symbol Device:C
- added J? (x3): DB9_Male_MountingHoles, Connector_Dsub:DSUB-9_Female_Horizontal_P2.77x2.84mm_EdgePinOffset7.70mm_Housed_MountingHolesOffset9.12mm, symbol Connector_Specialized:DB9_Male_MountingHoles
- added U? (x4): MAX3387EEUG, Package_SO:TSSOP-24_4.4x7.8mm_P0.65mm, symbol CommsCard:MAX3387EEUG
Connections:
- new net: J?.2, U?.18 (R1IN)
- new net: J?.3, U?.21 (T1OUT)
- new net: J?.2, U?.17 (R2IN)
- new net: J?.3, U?.20 (T2OUT)
- new net: J?.2, U?.16 (R3IN)
- new net: J?.3, U?.19 (T3OUT)
- new net: C?.1, U?.1 (C1+)
- new net: C?.1, U?.2 (V+)
- new net: C?.2, U?.3 (C1-)
- new net: C?.1, U?.4 (C2+)
- new net: C?.2, U?.5 (C2-)
- new net: C?.1, U?.6 (V-)
- new net +3V3: C?.1, U?.11 (GND), U?.15 (VL), U?.23 (VCC), U?.24 (~FORCEOFF)
- new net COMM1_RX: U?.14 (R1OUT)
- new net COMM1_TX: U?.7 (T1IN)
- new net COMM2_RX: U?.13 (R2OUT)
- new net COMM2_TX: U?.8 (T2IN)
- new net GND: C?.2, C?.2, C?.2, J?.5, J?.5, J?.5, U?.11 (GND)
- new net GNDPWR: J?.0 (PAD), J?.0 (PAD), J?.0 (PAD)
- new net HIGHRATE_RX: U?.12 (R3OUT)
- new net HIGHRATE_TX: U?.10 (T3IN)
- no-connect marks 0 -> 1
