File: design/Input.sch (KiCad schematic (older format))
At the start: 0 parts

Commit message: Adding Input Schematic
Parts:
- added C? (x10): 0u1F, Capacitors_SMD:C_0603, symbol Device:C
- added C? (x2): 4u7F, Capacitors_SMD:C_0603, symbol Device:C
- added C? (x2): 27pF, Capacitors_SMD:C_0603, symbol Device:C
- added C?: 3u3F, Capacitors_SMD:C_0603, symbol Device:C
- added L? (x2): 4u7H, Resistors_SMD:R_0603, symbol Device:L
- added R?: 12k, Resistors_SMD:R_0603, symbol Device:R
- added R?: 1k, symbol Device:R
- added R? (x8): 10k, Resistors_SMD:R_0603, symbol Device:R
- added R?: 2k2, Resistors_SMD:R_0603, symbol Device:R
- added U?: FT4232H, symbol Interface_USB:FT4232H
- added U?: 93C46B, Housings_SOIC:SOIC-8_3.9x4.9mm_Pitch1.27mm, symbol CommsCard:93CxxB
- added Y?: ABM8G, Crystals:Crystal_SMD_Abracon_ABM8G-4pin_3.2x2.5mm, symbol CommsCard:Crystal_GND24
Connections:
- net labels added: +1V8, 3V3, 5V, COMM1_RX, COMM1_TX, COMM2_RX, COMM2_TX, GND, HIGHRATE_RX, HIGHRATE_TX, IN_CHARGE, LOS_CLK, LOS_DATA, USB_DM, USB_DP, WD_TICKLE, ~PWREN
- wire segments 0 -> 159
- no-connect marks 0 -> 22

Commit message: adding power input connectors
Connections:
- net labels added: +3.3V, +5V
- net labels removed: 3V3, 5V
- wire segments 159 -> 162
Changed lines of the file:
@@
 Wire Wire Line
 	3350 3250 3300 3250
-Text HLabel 3300 3250 0    50   Input ~ 0
-3V3
 Wire Wire Line
 	1450 4800 1350 4800
-Text HLabel 1350 4800 0    50   Input ~ 0
-5V
 Wire Wire Line
 	3800 2750 3700 2750
@@
 	2850 3450 2850 3400
 Wire Wire Line
-	3800 3050 2850 3050
-Wire Wire Line
-	2850 3050 2850 3100
-Text HLabel 2800 1750 0    50   Input ~ 0
-3V3
+	3800 3050 3650 3050
 Wire Wire Line
 	3650 3250 3800 3250
@@
 Wire Wire Line
 	3350 2400 3350 2350
-Wire Wire Line
-	2800 1750 3050 1750
 $Comp
 L Device:C C?
@@
 	3600 1950 3800 1950
 Wire Wire Line
-	3050 2000 3050 1750
-Connection ~ 3050 1750
-Wire Wire Line
-	3050 1750 3800 1750
-Wire Wire Line
 	3350 2350 3050 2350
 Wire Wire Line
@@
 Wire Wire Line
 	3300 1400 3300 1300
-Text HLabel 1700 1150 0    50   Input ~ 0
-3V3
 Wire Wire Line
 	1700 1150 1950 1150
@@
 Wire Wire Line
 	5350 1400 5400 1400
-Text HLabel 5350 1300 1    50   Input ~ 0
-3V3
 Connection ~ 3950 1300
 Wire Wire Line
@@
 	6750 950  6750 850
 Connection ~ 6750 950
-Text HLabel 6750 850  1    50   Input ~ 0
-3V3
 Wire Wire Line
 	7400 1000 7400 950
@@
 Text HLabel 6250 3650 2    50   Output ~ 0
 COMM2_RX
-Text HLabel 3200 3750 1    50   Input ~ 0
-3V3
 Wire Wire Line
 	6200 4450 6250 4450
@@
 NoConn ~ 6200 5050
 Wire Wire Line
-	6650 2950 6750 2950
-Text HLabel 6750 2950 2    50   Input ~ 0
-3V3
-Wire Wire Line
-	6650 3850 6750 3850
-Text HLabel 6750 3850 2    50   Input ~ 0
-3V3
-Wire Wire Line
-	6650 4750 6750 4750
-Text HLabel 6750 4750 2    50   Input ~ 0
-3V3
+	6650 2950 6900 2950
+Wire Wire Line
+	6650 3850 6900 3850
+Wire Wire Line
+	6650 4750 6900 4750
 Wire Wire Line
 	6350 4750 6200 4750
@@
 Wire Wire Line
 	6850 5000 7100 5000
+$Comp
+L power:+1V8 #PWR?
+U 1 1 5A808A5A
+P 3600 1950
+F 0 "#PWR?" H 3600 1800 50  0001 C CNN
+F 1 "+1V8" H 3615 2123 50  0000 C CNN
+F 2 "" H 3600 1950 50  0001 C CNN
+F 3 "" H 3600 1950 50  0001 C CNN
+	1    3600 1950
+	1    0    0    -1
+$EndComp
+Connection ~ 3600 1950
+$Comp
+L power:+3.3V #PWR?
+U 1 1 5A808AF8
+P 3050 1700
+F 0 "#PWR?" H 3050 1550 50  0001 C CNN
+F 1 "+3.3V" H 3065 1873 50  0000 C CNN
+F 2 "" H 3050 1700 50  0001 C CNN
+F 3 "" H 3050 1700 50  0001 C CNN
+	1    3050 1700
+	1    0    0    -1
+$EndComp
+$Comp
+L power:+3.3V #PWR?
+U 1 1 5A80E9F1
+P 5350 1300
+F 0 "#PWR?" H 5350 1150 50  0001 C CNN
+F 1 "+3.3V" H 5365 1473 50  0000 C CNN
+F 2 "" H 5350 1300 50  0001 C CNN
+F 3 "" H 5350 1300 50  0001 C CNN
+	1    5350 1300
+	1    0    0    -1
+$EndComp
+$Comp
+L power:+3.3V #PWR?
+U 1 1 5A80EA7D
+P 1700 1150
+F 0 "#PWR?" H 1700 1000 50  0001 C CNN
+F 1 "+3.3V" H 1715 1323 50  0000 C CNN
+F 2 "" H 1700 1150 50  0001 C CNN
+F 3 "" H 1700 1150 50  0001 C CNN
+	1    1700 1150
+	1    0    0    -1
+$EndComp
+$Comp
+L power:+3.3V #PWR?
+U 1 1 5A814AA2
+P 6750 850
+F 0 "#PWR?" H 6750 700 50  0001 C CNN
+F 1 "+3.3V" H 6765 1023 50  0000 C CNN
+F 2 "" H 6750 850 50  0001 C CNN
+F 3 "" H 6750 850 50  0001 C CNN
+	1    6750 850
+	1    0    0    -1
+$EndComp
+$Comp
+L power:+3.3V #PWR?
+U 1 1 5A81AD3D
+P 6900 4750
+F 0 "#PWR?" H 6900 4600 50  0001 C CNN
+F 1 "+3.3V" H 6915 4923 50  0000 C CNN
+F 2 "" H 6900 4750 50  0001 C CNN
+F 3 "" H 6900 4750 50  0001 C CNN
+	1    6900 4750
+	1    0    0    -1
+$EndComp
+$Comp
+L power:+3.3V #PWR?
+U 1 1 5A820A99
+P 6900 3850
+F 0 "#PWR?" H 6900 3700 50  0001 C CNN
+F 1 "+3.3V" H 6915 4023 50  0000 C CNN
+F 2 "" H 6900 3850 50  0001 C CNN
+F 3 "" H 6900 3850 50  0001 C CNN
+	1    6900 3850
+	1    0    0    -1
+$EndComp
+$Comp
+L power:+3.3V #PWR?
+U 1 1 5A8267F5
+P 6900 2950
+F 0 "#PWR?" H 6900 2800 50  0001 C CNN
+F 1 "+3.3V" H 6915 3123 50  0000 C CNN
+F 2 "" H 6900 2950 50  0001 C CNN
+F 3 "" H 6900 2950 50  0001 C CNN
+	1    6900 2950
+	1    0    0    -1
+$EndComp
+$Comp
+L power:+3.3V #PWR?
+U 1 1 5A8409AC
+P 3200 3750
+F 0 "#PWR?" H 3200 3600 50  0001 C CNN
+F 1 "+3.3V" H 3215 3923 50  0000 C CNN
+F 2 "" H 3200 3750 50  0001 C CNN
+F 3 "" H 3200 3750 50  0001 C CNN
+	1    3200 3750
+	1    0    0    -1
+$EndComp
+$Comp
+L power:+5V #PWR?
+U 1 1 5A846AEB
+P 1350 4800
+F 0 "#PWR?" H 1350 4650 50  0001 C CNN
+F 1 "+5V" H 1365 4973 50  0000 C CNN
+F 2 "" H 1350 4800 50  0001 C CNN
+F 3 "" H 1350 4800 50  0001 C CNN
+	1    1350 4800
+	1    0    0    -1
+$EndComp
+$Comp
+L power:+3.3V #PWR?
+U 1 1 5A848044
+P 3300 3250
+F 0 "#PWR?" H 3300 3100 50  0001 C CNN
+F 1 "+3.3V" H 3315 3423 50  0000 C CNN
+F 2 "" H 3300 3250 50  0001 C CNN
+F 3 "" H 3300 3250 50  0001 C CNN
+	1    3300 3250
+	1    0    0    -1
+$EndComp
+Wire Wire Line
+	3650 3050 3650 2950
+Wire Wire Line
+	3650 2950 2850 2950
+Wire Wire Line
+	3750 1750 3750 1700
+Wire Wire Line
+	3750 1700 3050 1700
+Wire Wire Line
+	2850 2950 2850 3100
+Wire Wire Line
+	3750 1750 3800 1750
+Connection ~ 3050 1700
+Wire Wire Line
+	3050 1700 3050 2000
 $EndSCHEMATC

Commit message: Connecting LOS inside FC connection
Parts:
- added J?: Conn_01x03, Pin_Headers:Pin_Header_Straight_1x03_Pitch2.54mm, symbol Connector_Generic:Conn_01x03
Connections:
- net labels added: LOS
- net labels removed: LOS_CLK, LOS_DATA
- wire segments 162 -> 169
Changed lines of the file:
@@
 $Descr A4 11693 8268
 encoding utf-8
-Sheet 6 7
+Sheet 6 8
 Title ""
 Date ""
@@
 	1    0    0    -1
 $EndComp
-Wire Wire Line
-	6200 1750 6250 1750
-Wire Wire Line
-	6200 1850 6250 1850
-Text HLabel 6250 1750 2    50   Output ~ 0
-LOS_CLK
-Text HLabel 6250 1850 2    50   Output ~ 0
-LOS_DATA
 NoConn ~ 6200 1950
 NoConn ~ 6200 2050
@@
 Wire Wire Line
 	3050 1700 3050 2000
+$Sheet
+S 8100 1550 950  550
+U 5A7DC371
+F0 "LOSComms" 50
+F1 "LOSComms.sch" 50
+F2 "DATA" I L 8100 1850 50
+F3 "RNRZ-L" O R 9050 1750 50
+F4 "CLK" I L 8100 1750 50
+F5 "BIPHASE" O R 9050 1850 50
+$EndSheet
+Wire Wire Line
+	6200 1750 8100 1750
+Wire Wire Line
+	6200 1850 8100 1850
+$Comp
+L Connector_Generic:Conn_01x03 J?
+U 1 1 5A806EE1
+P 9650 1800
+F 0 "J?" H 9730 1842 50  0000 L CNN
+F 1 "Conn_01x03" H 9730 1751 50  0000 L CNN
+F 2 "Pin_Headers:Pin_Header_Straight_1x03_Pitch2.54mm" H 9650 1800 50  0001 C CNN
+F 3 "https://cdn.harwin.com/pdfs/M20-999.pdf" H 9650 1800 50  0001 C CNN
+F 4 "M20-9990345" H 9650 1800 50  0001 C CNN "mpn"
+	1    9650 1800
+	1    0    0    -1
+$EndComp
+Wire Wire Line
+	9450 1700 9350 1700
+Wire Wire Line
+	9350 1700 9350 1750
+Wire Wire Line
+	9350 1750 9050 1750
+Wire Wire Line
+	9050 1850 9350 1850
+Wire Wire Line
+	9350 1850 9350 1900
+Wire Wire Line
+	9350 1900 9450 1900
+Wire Wire Line
+	9450 1800 10400 1800
+Text HLabel 10400 1800 2    50   Output ~ 0
+LOS
 $EndSCHEMATC

Commit message: Finished ERC
Parts:
- gave numbers to parts that had none: 32
Connections:
- net labels added: 1V8
- net labels removed: +1V8

Commit message: Adding LED Indicator for tx/rx
Parts:
- added D501, D502, D503: WP130WDT/EGW, LED_THT:LED_D5.0mm-3, symbol Device:LED_Dual_ACA
- added R512: 10k, Resistors_SMD:R_0603, symbol Device:R
- added RN501: 330R, ResistorArray:R_Array_Convex_8x0402, symbol Device:R_Pack08
- added U503: 74HC595, ResistorArray:R_Array_Convex_8x0402, symbol Logic_74xx:74HC595
Connections:
- net labels added: EECLK, EECS, EEDATA
- wire segments 169 -> 206
- no-connect marks 22 -> 25

Commit message: Swapping FT4232 for VQFN and finalizing mpns
Parts:
- R505: value 1k -> 10k; footprint (none) -> Resistors_SMD:R_0603; mpn (none) -> CRG0603F1K0
- U502: footprint (none) -> Package_DFN_QFN:QFN-56-1EP_8x8mm_P0.5mm_EP4.5x5.2mm; symbol Interface_USB:FT4232H -> CommsCard:FT4232H-56Q; mpn (none) -> FT4232H-56Q-TRAY
- U503: footprint ResistorArray:R_Array_Convex_8x0402 -> Package_SO:TSSOP-16_4.4x5mm_P0.65mm; mpn (none) -> 74HC595PW,118
Connections:
- wire segments 206 -> 197
Changed lines of the file:
@@
 $EndDescr
 $Comp
-L Interface_USB:FT4232H U502
+L CommsCard:FT4232H-56Q U502
 U 1 1 5A7727AC
 P 5000 3650
@@
 F 0 "U702" H 5000 4000 50  0000 C CNN
 F 1 "FT4232H" H 5000 3850 50  0000 C CNN
-F 2 "" H 5000 3650 50  0001 C CNN
-F 3 "" H 5000 3650 50  0001 C CNN
+F 2 "Package_DFN_QFN:QFN-56-1EP_8x8mm_P0.5mm_EP4.5x5.2mm" H 5000 3650 50  0001 C CNN
+F 3 "http://www.ftdichip.com/Support/Documents/DataSheets/ICs/DS_FT4232H.pdf" H 5000 3650 50  0001 C CNN
+F 4 "FT4232H-56Q-TRAY" H 5000 3650 50  0001 C CNN "mpn"
 	1    5000 3650
 	1    0    0    -1
@@
 $EndComp
 $Comp
-L Device:R R505
-U 1 1 5A7731D9
-P 3500 3250
-AR Path="/5A78E64E/5A7731D9" Ref="R505"  Part="1"
-AR Path="/5A78E661/5A7731D9" Ref="R705"  Part="1"
-F 0 "R705" V 3600 3250 50  0000 C CNN
-F 1 "1k" V 3384 3250 50  0000 C CNN
-F 2 "" V 3430 3250 50  0001 C CNN
-F 3 "~" H 3500 3250 50  0001 C CNN
-	1    3500 3250
-	0    -1   1    0
-$EndComp
-$Comp
 L CommsCard:93CxxB U501
 U 1 1 5A7734DE
@@
 	3800 5750 4400 5750
 Connection ~ 4400 5750
-Wire Wire Line
-	4400 5750 4600 5750
-Connection ~ 4600 5750
-Wire Wire Line
-	4600 5750 4700 5750
 Connection ~ 4700 5750
-Wire Wire Line
-	4700 5750 4800 5750
-Connection ~ 4800 5750
-Wire Wire Line
-	4800 5750 4900 5750
 Connection ~ 4900 5750
-Wire Wire Line
-	4900 5750 5000 5750
-Connection ~ 5000 5750
-Wire Wire Line
-	5000 5750 5100 5750
 Connection ~ 5100 5750
-Wire Wire Line
-	5100 5750 5200 5750
-Connection ~ 5200 5750
-Wire Wire Line
-	5200 5750 5300 5750
 Wire Wire Line
 	4400 6000 4400 5750
@@
 	3300 1300 3050 1300
 Wire Wire Line
-	5000 1450 5000 1400
-Wire Wire Line
-	5000 1400 4900 1400
-Wire Wire Line
 	4800 1400 4800 1450
 Wire Wire Line
@@
 	5200 1400 5300 1400
 Wire Wire Line
-	5500 1400 5500 1450
-Wire Wire Line
 	5400 1450 5400 1400
-Connection ~ 5400 1400
-Wire Wire Line
-	5400 1400 5500 1400
 Wire Wire Line
 	5300 1400 5300 1450
 Connection ~ 5300 1400
 Wire Wire Line
-	5300 1400 5350 1400
-Wire Wire Line
-	5350 1400 5350 1300
-Connection ~ 5350 1400
-Wire Wire Line
-	5350 1400 5400 1400
+	5300 1400 5300 1300
+Wire Wire Line
+	5300 1400 5400 1400
 Connection ~ 3950 1300
 Wire Wire Line
@@
 L power:+3.3V #PWR0512
 U 1 1 5A80E9F1
-P 5350 1300
+P 5300 1300
 AR Path="/5A78E64E/5A80E9F1" Ref="#PWR0512"  Part="1"
 AR Path="/5A78E661/5A80E9F1" Ref="#PWR0712"  Part="1"
-F 0 "#PWR0712" H 5350 1150 50  0001 C CNN
-F 1 "+3.3V" H 5365 1473 50  0000 C CNN
-F 2 "" H 5350 1300 50  0001 C CNN
-F 3 "" H 5350 1300 50  0001 C CNN
-	1    5350 1300
+F 0 "#PWR0712" H 5300 1150 50  0001 C CNN
+F 1 "+3.3V" H 5315 1473 50  0000 C CNN
+F 2 "" H 5300 1300 50  0001 C CNN
+F 3 "" H 5300 1300 50  0001 C CNN
+	1    5300 1300
 	1    0    0    -1
 $EndComp
@@
 F 0 "U703" H 9050 4400 50  0000 C CNN
 F 1 "74HC595" H 9050 4300 50  0000 C CNN
-F 2 "ResistorArray:R_Array_Convex_8x0402" H 8850 3700 50  0001 C CNN
-F 3 "http://www.nxp.com/documents/data_sheet/74HC_HCT595.pdf" H 8850 3700 50  0001 C CNN
-F 4 "~" H 8850 3700 50  0001 C CNN "mpn"
+F 2 "Package_SO:TSSOP-16_4.4x5mm_P0.65mm" H 8850 3700 50  0001 C CNN
+F 3 "https://assets.nexperia.com/documents/data-sheet/74HC_HCT595.pdf" H 8850 3700 50  0001 C CNN
+F 4 "74HC595PW,118" H 8850 3700 50  0001 C CNN "mpn"
 	1    8850 3700
 	1    0    0    -1
@@
 Wire Wire Line
 	7850 3900 8300 3900
+Wire Wire Line
+	4400 5750 4700 5750
+Wire Wire Line
+	4700 5750 4900 5750
+Wire Wire Line
+	4900 5750 5100 5750
+Wire Wire Line
+	5100 5750 5300 5750
+$Comp
+L Device:R R505
+U 1 1 5A88BF7E
+P 3500 3250
+AR Path="/5A78E64E/5A88BF7E" Ref="R505"  Part="1"
+AR Path="/5A78E661/5A88BF7E" Ref="R705"  Part="1"
+F 0 "R705" V 3400 3250 50  0000 C CNN
+F 1 "10k" V 3600 3250 50  0000 C CNN
+F 2 "Resistors_SMD:R_0603" V 3430 3250 50  0001 C CNN
+F 3 "http://www.te.com/commerce/DocumentDelivery/DDEController?Action=srchrtrv&DocNm=1773204&DocType=DS&DocLang=English" H 3500 3250 50  0001 C CNN
+F 4 "CRG0603F1K0" H 3500 3250 50  0001 C CNN "mpn"
+	1    3500 3250
+	0    -1   1    0
+$EndComp
 $EndSCHEMATC
