File: design/Input.sch (KiCad schematic (older format))
At the start: 38 parts, among them J501 Conn_01x03, U501 93C46B, U502 FT4232H, U503 74HC595, Y501 ABM8G

Commit message: Updating schematic for layout
Parts:
- removed C502, C505: 27pF, Capacitors_SMD:C_0603, symbol Device:C
- removed Y501: ABM8G, Crystals:Crystal_SMD_Abracon_ABM8G-4pin_3.2x2.5mm, symbol CommsCard:Crystal_GND24
- added C516: 10nF, Capacitor_SMD:C_0603_1608Metric, symbol Device:C
- added R513: 10k, Resistor_SMD:R_0603_1608Metric, symbol Device:R
- added X501: ASEMB-12MHz, Oscillator:Oscillator_SMD_Abracon_ASE-4Pin_3.2x2.5mm, symbol Oscillator:ASE-xxxMHz
- C501, C503, C507: footprint Capacitors_SMD:C_0603 -> Capacitor_SMD:C_0603_1608Metric
- C504, C506, C508, C509, C510, C511, C512, C513, C514, C515: footprint Capacitors_SMD:C_0603 -> Capacitor_SMD:C_0603_1608Metric; mpn CL10F104ZB8NNNC -> CL10B104KO8WPNC
- J501: footprint Pin_Headers:Pin_Header_Straight_1x03_Pitch2.54mm -> Connector_PinHeader_2.54mm:PinHeader_1x03_P2.54mm_Vertical
- L501, L502, R501, R502, R503, R504: footprint Resistors_SMD:R_0603 -> Resistor_SMD:R_0603_1608Metric
- R505, R506, R507, R508, R509, R510, R511, R512: footprint Resistors_SMD:R_0603 -> Resistor_SMD:R_0603_1608Metric; mpn CRG0603F1K0 -> CRG0603J10K
- U501: footprint Housings_SOIC:SOIC-8_3.9x4.9mm_Pitch1.27mm -> Package_SO:SOIC-8_3.9x4.9mm_P1.27mm
- U503: value 74HC595 -> 74LV595; mpn 74HC595PW,118 -> SN74LV595APWR
Connections:
- wire segments 197 -> 184
- no-connect marks 25 -> 26
Other:
- moved on the sheet: U501

Commit message: Switching PLL inductor
Parts:
- removed L501: 4u7H, Resistor_SMD:R_0603_1608Metric, symbol Device:L
- added L501: 4u7H, Resistor_SMD:R_1210_3225Metric, symbol Device:L_Core_Iron
- L502: footprint Resistor_SMD:R_0603_1608Metric -> Resistor_SMD:R_1210_3225Metric; symbol Device:L -> Device:L_Core_Iron; mpn AIML-0603-4R7K-T -> 1277AS-H-4R7M=P2
Changed lines of the file:
@@
 $EndComp
 $Comp
-L Device:L L501
-U 1 1 5A772E6B
-P 2150 1000
-AR Path="/5A78E64E/5A772E6B" Ref="L501"  Part="1"
-AR Path="/5A78E661/5A772E6B" Ref="L701"  Part="1"
-F 0 "L501" V 1972 1000 50  0000 C CNN
-F 1 "4u7H" V 2063 1000 50  0000 C CNN
-F 2 "Resistor_SMD:R_0603_1608Metric" H 2150 1000 50  0001 C CNN
-F 3 "http://www.abracon.com/Magnetics/new/AIML-0603.pdf" H 2150 1000 50  0001 C CNN
-F 4 "AIML-0603-4R7K-T" H 2150 1000 50  0001 C CNN "mpn"
-	1    2150 1000
-	0    1    1    0
-$EndComp
-$Comp
-L Device:L L502
+L Device:L_Core_Iron L502
 U 1 1 5A772FF6
 P 2150 1300
@@
 F 0 "L502" V 1972 1300 50  0000 C CNN
 F 1 "4u7H" V 2063 1300 50  0000 C CNN
-F 2 "Resistor_SMD:R_0603_1608Metric" H 2150 1300 50  0001 C CNN
-F 3 "http://www.abracon.com/Magnetics/new/AIML-0603.pdf" H 2150 1300 50  0001 C CNN
-F 4 "AIML-0603-4R7K-T" H 2150 1300 50  0001 C CNN "mpn"
+F 2 "Resistor_SMD:R_1210_3225Metric" H 2150 1300 50  0001 C CNN
+F 3 "https://www.murata.com/~/media/webrenewal/products/inductor/chip/tokoproducts/wirewoundmetalalloychiptype/m_dfe322512c.ashx" H 2150 1300 50  0001 C CNN
+F 4 "1277AS-H-4R7M=P2" H 2150 1300 50  0001 C CNN "mpn"
 	1    2150 1300
 	0    1    1    0
@@
 AR Path="/5A78E64E/5A7760FD" Ref="#PWR0502"  Part="1"
 AR Path="/5A78E661/5A7760FD" Ref="#PWR0702"  Part="1"
-F 0 "#PWR0702" H 1400 4650 50  0001 C CNN
+F 0 "#PWR0502" H 1400 4650 50  0001 C CNN
 F 1 "GND" H 1405 4727 50  0000 C CNN
 F 2 "" H 1400 4900 50  0001 C CNN
@@
 AR Path="/5A78E64E/5A77612B" Ref="#PWR0511"  Part="1"
 AR Path="/5A78E661/5A77612B" Ref="#PWR0711"  Part="1"
-F 0 "#PWR0711" H 4400 5750 50  0001 C CNN
+F 0 "#PWR0511" H 4400 5750 50  0001 C CNN
 F 1 "GND" H 4405 5827 50  0000 C CNN
 F 2 "" H 4400 6000 50  0001 C CNN
@@
 AR Path="/5A78E64E/5A78FA4C" Ref="#PWR0504"  Part="1"
 AR Path="/5A78E661/5A78FA4C" Ref="#PWR0704"  Part="1"
-F 0 "#PWR0704" H 2850 3200 50  0001 C CNN
+F 0 "#PWR0504" H 2850 3200 50  0001 C CNN
 F 1 "GND" H 2855 3277 50  0000 C CNN
 F 2 "" H 2850 3450 50  0001 C CNN
@@
 AR Path="/5A78E64E/5A79780B" Ref="#PWR0510"  Part="1"
 AR Path="/5A78E661/5A79780B" Ref="#PWR0710"  Part="1"
-F 0 "#PWR0710" H 3350 2150 50  0001 C CNN
+F 0 "#PWR0510" H 3350 2150 50  0001 C CNN
 F 1 "GND" H 3355 2227 50  0000 C CNN
 F 2 "" H 3350 2400 50  0001 C CNN
@@
 AR Path="/5A78E64E/5A7A5A9C" Ref="#PWR0508"  Part="1"
 AR Path="/5A78E661/5A7A5A9C" Ref="#PWR0708"  Part="1"
-F 0 "#PWR0708" H 3300 1150 50  0001 C CNN
+F 0 "#PWR0508" H 3300 1150 50  0001 C CNN
 F 1 "GND" H 3305 1227 50  0000 C CNN
 F 2 "" H 3300 1400 50  0001 C CNN
@@
 AR Path="/5A78E64E/5A7DFDD9" Ref="#PWR0517"  Part="1"
 AR Path="/5A78E661/5A7DFDD9" Ref="#PWR0717"  Part="1"
-F 0 "#PWR0717" H 7400 1250 50  0001 C CNN
+F 0 "#PWR0517" H 7400 1250 50  0001 C CNN
 F 1 "GND" H 7405 1327 50  0000 C CNN
 F 2 "" H 7400 1500 50  0001 C CNN
@@
 AR Path="/5A78E64E/5A808AF8" Ref="#PWR0506"  Part="1"
 AR Path="/5A78E661/5A808AF8" Ref="#PWR0706"  Part="1"
-F 0 "#PWR0706" H 3050 1550 50  0001 C CNN
+F 0 "#PWR0506" H 3050 1550 50  0001 C CNN
 F 1 "+3.3V" H 3065 1873 50  0000 C CNN
 F 2 "" H 3050 1700 50  0001 C CNN
@@
 AR Path="/5A78E64E/5A80E9F1" Ref="#PWR0512"  Part="1"
 AR Path="/5A78E661/5A80E9F1" Ref="#PWR0712"  Part="1"
-F 0 "#PWR0712" H 5300 1150 50  0001 C CNN
+F 0 "#PWR0512" H 5300 1150 50  0001 C CNN
 F 1 "+3.3V" H 5315 1473 50  0000 C CNN
 F 2 "" H 5300 1300 50  0001 C CNN
@@
 AR Path="/5A78E64E/5A80EA7D" Ref="#PWR0503"  Part="1"
 AR Path="/5A78E661/5A80EA7D" Ref="#PWR0703"  Part="1"
-F 0 "#PWR0703" H 1700 1000 50  0001 C CNN
+F 0 "#PWR0503" H 1700 1000 50  0001 C CNN
 F 1 "+3.3V" H 1715 1323 50  0000 C CNN
 F 2 "" H 1700 1150 50  0001 C CNN
@@
 AR Path="/5A78E64E/5A814AA2" Ref="#PWR0513"  Part="1"
 AR Path="/5A78E661/5A814AA2" Ref="#PWR0713"  Part="1"
-F 0 "#PWR0713" H 6750 700 50  0001 C CNN
+F 0 "#PWR0513" H 6750 700 50  0001 C CNN
 F 1 "+3.3V" H 6765 1023 50  0000 C CNN
 F 2 "" H 6750 850 50  0001 C CNN
@@
 AR Path="/5A78E64E/5A81AD3D" Ref="#PWR0516"  Part="1"
 AR Path="/5A78E661/5A81AD3D" Ref="#PWR0716"  Part="1"
-F 0 "#PWR0716" H 6900 4600 50  0001 C CNN
+F 0 "#PWR0516" H 6900 4600 50  0001 C CNN
 F 1 "+3.3V" H 6915 4923 50  0000 C CNN
 F 2 "" H 6900 4750 50  0001 C CNN
@@
 AR Path="/5A78E64E/5A820A99" Ref="#PWR0515"  Part="1"
 AR Path="/5A78E661/5A820A99" Ref="#PWR0715"  Part="1"
-F 0 "#PWR0715" H 6900 3700 50  0001 C CNN
+F 0 "#PWR0515" H 6900 3700 50  0001 C CNN
 F 1 "+3.3V" H 6915 4023 50  0000 C CNN
 F 2 "" H 6900 3850 50  0001 C CNN
@@
 AR Path="/5A78E64E/5A8267F5" Ref="#PWR0514"  Part="1"
 AR Path="/5A78E661/5A8267F5" Ref="#PWR0714"  Part="1"
-F 0 "#PWR0714" H 6900 2800 50  0001 C CNN
+F 0 "#PWR0514" H 6900 2800 50  0001 C CNN
 F 1 "+3.3V" H 6915 3123 50  0000 C CNN
 F 2 "" H 6900 2950 50  0001 C CNN
@@
 AR Path="/5A78E64E/5A8409AC" Ref="#PWR0507"  Part="1"
 AR Path="/5A78E661/5A8409AC" Ref="#PWR0707"  Part="1"
-F 0 "#PWR0707" H 3200 3600 50  0001 C CNN
+F 0 "#PWR0507" H 3200 3600 50  0001 C CNN
 F 1 "+3.3V" H 3215 3923 50  0000 C CNN
 F 2 "" H 3200 3750 50  0001 C CNN
@@
 AR Path="/5A78E64E/5A846AEB" Ref="#PWR0501"  Part="1"
 AR Path="/5A78E661/5A846AEB" Ref="#PWR0701"  Part="1"
-F 0 "#PWR0701" H 1350 4200 50  0001 C CNN
+F 0 "#PWR0501" H 1350 4200 50  0001 C CNN
 F 1 "+5V" H 1365 4523 50  0000 C CNN
 F 2 "" H 1350 4350 50  0001 C CNN
@@
 AR Path="/5A78E64E/5A848044" Ref="#PWR0509"  Part="1"
 AR Path="/5A78E661/5A848044" Ref="#PWR0709"  Part="1"
-F 0 "#PWR0709" H 3300 3100 50  0001 C CNN
+F 0 "#PWR0509" H 3300 3100 50  0001 C CNN
 F 1 "+3.3V" H 3315 3423 50  0000 C CNN
 F 2 "" H 3300 3250 50  0001 C CNN
@@
 AR Path="/5A78E64E/5A8B20A8" Ref="#FLG0501"  Part="1"
 AR Path="/5A78E661/5A8B20A8" Ref="#FLG0701"  Part="1"
-F 0 "#FLG0701" H 2600 1075 50  0001 C CNN
+F 0 "#FLG0501" H 2600 1075 50  0001 C CNN
 F 1 "PWR_FLAG" H 2600 1174 50  0000 C CNN
 F 2 "" H 2600 1000 50  0001 C CNN
@@
 AR Path="/5A78E64E/5A83C347" Ref="#PWR0521"  Part="1"
 AR Path="/5A78E661/5A83C347" Ref="#PWR0721"  Part="1"
-F 0 "#PWR0721" H 10850 4250 50  0001 C CNN
+F 0 "#PWR0521" H 10850 4250 50  0001 C CNN
 F 1 "GND" H 10855 4327 50  0000 C CNN
 F 2 "" H 10850 4500 50  0001 C CNN
@@
 AR Path="/5A78E64E/5A878935" Ref="#PWR0519"  Part="1"
 AR Path="/5A78E661/5A878935" Ref="#PWR0719"  Part="1"
-F 0 "#PWR0719" H 8850 2850 50  0001 C CNN
+F 0 "#PWR0519" H 8850 2850 50  0001 C CNN
 F 1 "+3.3V" H 8865 3173 50  0000 C CNN
 F 2 "" H 8850 3000 50  0001 C CNN
@@
 AR Path="/5A78E64E/5A878991" Ref="#PWR0520"  Part="1"
 AR Path="/5A78E661/5A878991" Ref="#PWR0720"  Part="1"
-F 0 "#PWR0720" H 8850 4250 50  0001 C CNN
+F 0 "#PWR0520" H 8850 4250 50  0001 C CNN
 F 1 "GND" H 8855 4327 50  0000 C CNN
 F 2 "" H 8850 4500 50  0001 C CNN
@@
 AR Path="/5A78E64E/5A89E551" Ref="#PWR0518"  Part="1"
 AR Path="/5A78E661/5A89E551" Ref="#PWR0718"  Part="1"
-F 0 "#PWR0718" H 7850 3300 50  0001 C CNN
+F 0 "#PWR0518" H 7850 3300 50  0001 C CNN
 F 1 "+3.3V" H 7865 3623 50  0000 C CNN
 F 2 "" H 7850 3450 50  0001 C CNN
@@
 AR Path="/5A78E64E/5A92C971" Ref="#PWR01"  Part="1"
 AR Path="/5A78E661/5A92C971" Ref="#PWR04"  Part="1"
-F 0 "#PWR04" H 2000 5300 50  0001 C CNN
+F 0 "#PWR01" H 2000 5300 50  0001 C CNN
 F 1 "GND" H 2005 5377 50  0000 C CNN
 F 2 "" H 2000 5550 50  0001 C CNN
@@
 AR Path="/5A78E64E/5A92C9CE" Ref="#PWR02"  Part="1"
 AR Path="/5A78E661/5A92C9CE" Ref="#PWR05"  Part="1"
-F 0 "#PWR05" H 2800 5600 50  0001 C CNN
+F 0 "#PWR02" H 2800 5600 50  0001 C CNN
 F 1 "GND" H 2805 5677 50  0000 C CNN
 F 2 "" H 2800 5850 50  0001 C CNN
@@
 AR Path="/5A78E64E/5A949389" Ref="#PWR03"  Part="1"
 AR Path="/5A78E661/5A949389" Ref="#PWR06"  Part="1"
-F 0 "#PWR06" H 2800 4950 50  0001 C CNN
+F 0 "#PWR03" H 2800 4950 50  0001 C CNN
 F 1 "+3.3V" H 2815 5273 50  0000 C CNN
 F 2 "" H 2800 5100 50  0001 C CNN
@@
 Wire Wire Line
 	3700 4850 3800 4850
+$Comp
+L Device:L_Core_Iron L501
+U 1 1 5A852718
+P 2150 1000
+AR Path="/5A78E64E/5A852718" Ref="L501"  Part="1"
+AR Path="/5A78E661/5A852718" Ref="L701"  Part="1"
+F 0 "L501" V 1972 1000 50  0000 C CNN
+F 1 "4u7H" V 2063 1000 50  0000 C CNN
+F 2 "Resistor_SMD:R_1210_3225Metric" H 2150 1000 50  0001 C CNN
+F 3 "https://www.murata.com/~/media/webrenewal/products/inductor/chip/tokoproducts/wirewoundmetalalloychiptype/m_dfe322512c.ashx" H 2150 1000 50  0001 C CNN
+F 4 "1277AS-H-4R7M=P2" H 2150 1000 50  0001 C CNN "mpn"
+	1    2150 1000
+	0    1    1    0
+$EndComp
 $EndSCHEMATC

Commit message: Correcting PLL wiring
Connections:
- wire segments 184 -> 186
Changed lines of the file:
@@
 L Device:C C506
 U 1 1 5A772A13
-P 3500 1150
+P 2500 1550
 AR Path="/5A78E64E/5A772A13" Ref="C506"  Part="1"
 AR Path="/5A78E661/5A772A13" Ref="C706"  Part="1"
-F 0 "C506" H 3615 1196 50  0000 L CNN
-F 1 "0u1F" H 3615 1105 50  0000 L CNN
-F 2 "Capacitor_SMD:C_0603_1608Metric" H 3538 1000 50  0001 C CNN
-F 3 "http://www.samsungsem.com/kr/support/product-search/mlcc/CL10B104KO8WPNC.jsp" H 3500 1150 50  0001 C CNN
-F 4 "CL10B104KO8WPNC" H 3500 1150 50  0001 C CNN "mpn"
-	1    3500 1150
+F 0 "C506" H 2615 1596 50  0000 L CNN
+F 1 "0u1F" H 2615 1505 50  0000 L CNN
+F 2 "Capacitor_SMD:C_0603_1608Metric" H 2538 1400 50  0001 C CNN
+F 3 "http://www.samsungsem.com/kr/support/product-search/mlcc/CL10B104KO8WPNC.jsp" H 2500 1550 50  0001 C CNN
+F 4 "CL10B104KO8WPNC" H 2500 1550 50  0001 C CNN "mpn"
+	1    2500 1550
 	1    0    0    -1
 $EndComp
@@
 L Device:C C503
 U 1 1 5A772A39
-P 3050 1150
+P 1900 1200
 AR Path="/5A78E64E/5A772A39" Ref="C503"  Part="1"
 AR Path="/5A78E661/5A772A39" Ref="C703"  Part="1"
-F 0 "C503" H 3165 1196 50  0000 L CNN
-F 1 "4u7F" H 3165 1105 50  0000 L CNN
-F 2 "Capacitor_SMD:C_0603_1608Metric" H 3088 1000 50  0001 C CNN
-F 3 "http://www.samsungsem.com/kr/support/product-search/mlcc/CL10A475KQ8NNNC.jsp" H 3050 1150 50  0001 C CNN
-F 4 "CL10A475KQ8NNNC" H 3050 1150 50  0001 C CNN "mpn"
-	1    3050 1150
+F 0 "C503" H 2015 1246 50  0000 L CNN
+F 1 "4u7F" H 2015 1155 50  0000 L CNN
+F 2 "Capacitor_SMD:C_0603_1608Metric" H 1938 1050 50  0001 C CNN
+F 3 "http://www.samsungsem.com/kr/support/product-search/mlcc/CL10A475KQ8NNNC.jsp" H 1900 1200 50  0001 C CNN
+F 4 "CL10A475KQ8NNNC" H 1900 1200 50  0001 C CNN "mpn"
+	1    1900 1200
 	1    0    0    -1
 $EndComp
@@
 L Device:C C501
 U 1 1 5A772A65
-P 2600 1150
+P 2050 1550
 AR Path="/5A78E64E/5A772A65" Ref="C501"  Part="1"
 AR Path="/5A78E661/5A772A65" Ref="C701"  Part="1"
-F 0 "C501" H 2715 1196 50  0000 L CNN
-F 1 "4u7F" H 2715 1105 50  0000 L CNN
-F 2 "Capacitor_SMD:C_0603_1608Metric" H 2638 1000 50  0001 C CNN
-F 3 "http://www.samsungsem.com/kr/support/product-search/mlcc/CL10A475KQ8NNNC.jsp" H 2600 1150 50  0001 C CNN
-F 4 "CL10A475KQ8NNNC" H 2600 1150 50  0001 C CNN "mpn"
-	1    2600 1150
+F 0 "C501" H 2165 1596 50  0000 L CNN
+F 1 "4u7F" H 2165 1505 50  0000 L CNN
+F 2 "Capacitor_SMD:C_0603_1608Metric" H 2088 1400 50  0001 C CNN
+F 3 "http://www.samsungsem.com/kr/support/product-search/mlcc/CL10A475KQ8NNNC.jsp" H 2050 1550 50  0001 C CNN
+F 4 "CL10A475KQ8NNNC" H 2050 1550 50  0001 C CNN "mpn"
+	1    2050 1550
 	1    0    0    -1
 $EndComp
@@
 L Device:C C508
 U 1 1 5A772AC3
-P 3950 1150
+P 2400 1200
 AR Path="/5A78E64E/5A772AC3" Ref="C508"  Part="1"
 AR Path="/5A78E661/5A772AC3" Ref="C708"  Part="1"
-F 0 "C508" H 4065 1196 50  0000 L CNN
-F 1 "0u1F" H 4065 1105 50  0000 L CNN
-F 2 "Capacitor_SMD:C_0603_1608Metric" H 3988 1000 50  0001 C CNN
-F 3 "http://www.samsungsem.com/kr/support/product-search/mlcc/CL10B104KO8WPNC.jsp" H 3950 1150 50  0001 C CNN
-F 4 "CL10B104KO8WPNC" H 3950 1150 50  0001 C CNN "mpn"
-	1    3950 1150
+F 0 "C508" H 2515 1246 50  0000 L CNN
+F 1 "0u1F" H 2515 1155 50  0000 L CNN
+F 2 "Capacitor_SMD:C_0603_1608Metric" H 2438 1050 50  0001 C CNN
+F 3 "http://www.samsungsem.com/kr/support/product-search/mlcc/CL10B104KO8WPNC.jsp" H 2400 1200 50  0001 C CNN
+F 4 "CL10B104KO8WPNC" H 2400 1200 50  0001 C CNN "mpn"
+	1    2400 1200
 	1    0    0    -1
 $EndComp
@@
 L Device:L_Core_Iron L502
 U 1 1 5A772FF6
-P 2150 1300
+P 1600 1400
 AR Path="/5A78E64E/5A772FF6" Ref="L502"  Part="1"
 AR Path="/5A78E661/5A772FF6" Ref="L702"  Part="1"
-F 0 "L502" V 1972 1300 50  0000 C CNN
-F 1 "4u7H" V 2063 1300 50  0000 C CNN
-F 2 "Resistor_SMD:R_1210_3225Metric" H 2150 1300 50  0001 C CNN
-F 3 "https://www.murata.com/~/media/webrenewal/products/inductor/chip/tokoproducts/wirewoundmetalalloychiptype/m_dfe322512c.ashx" H 2150 1300 50  0001 C CNN
-F 4 "1277AS-H-4R7M=P2" H 2150 1300 50  0001 C CNN "mpn"
-	1    2150 1300
+F 0 "L502" V 1422 1400 50  0000 C CNN
+F 1 "4u7H" V 1513 1400 50  0000 C CNN
+F 2 "Resistor_SMD:R_1210_3225Metric" H 1600 1400 50  0001 C CNN
+F 3 "https://www.murata.com/~/media/webrenewal/products/inductor/chip/tokoproducts/wirewoundmetalalloychiptype/m_dfe322512c.ashx" H 1600 1400 50  0001 C CNN
+F 4 "1277AS-H-4R7M=P2" H 1600 1400 50  0001 C CNN "mpn"
+	1    1600 1400
 	0    1    1    0
 $EndComp
@@
 L power:GND #PWR0508
 U 1 1 5A7A5A9C
-P 3300 1400
+P 2050 1850
 AR Path="/5A78E64E/5A7A5A9C" Ref="#PWR0508"  Part="1"
 AR Path="/5A78E661/5A7A5A9C" Ref="#PWR0708"  Part="1"
-F 0 "#PWR0508" H 3300 1150 50  0001 C CNN
-F 1 "GND" H 3305 1227 50  0000 C CNN
-F 2 "" H 3300 1400 50  0001 C CNN
-F 3 "" H 3300 1400 50  0001 C CNN
-	1    3300 1400
-	1    0    0    -1
-$EndComp
-Wire Wire Line
-	3300 1400 3300 1300
-Wire Wire Line
-	1700 1150 1950 1150
-Wire Wire Line
-	2000 1300 1950 1300
-Wire Wire Line
-	1950 1300 1950 1150
-Wire Wire Line
-	1950 1000 2000 1000
-Connection ~ 1950 1150
-Wire Wire Line
-	1950 1150 1950 1000
-Wire Wire Line
-	2300 1000 2600 1000
+F 0 "#PWR0508" H 2050 1600 50  0001 C CNN
+F 1 "GND" H 2055 1677 50  0000 C CNN
+F 2 "" H 2050 1850 50  0001 C CNN
+F 3 "" H 2050 1850 50  0001 C CNN
+	1    2050 1850
+	1    0    0    -1
+$EndComp
+Wire Wire Line
+	1150 1200 1400 1200
+Wire Wire Line
+	1450 1400 1400 1400
+Wire Wire Line
+	1400 1400 1400 1200
+Wire Wire Line
+	1400 1000 1450 1000
+Connection ~ 1400 1200
+Wire Wire Line
+	1400 1200 1400 1000
+Wire Wire Line
+	1750 1000 1900 1000
 Wire Wire Line
 	4600 1000 4600 1450
-Connection ~ 2600 1000
-Wire Wire Line
-	2600 1000 3050 1000
-Connection ~ 3050 1000
-Wire Wire Line
-	4500 1450 4500 1300
-Connection ~ 2600 1300
-Wire Wire Line
-	2600 1300 2300 1300
-Connection ~ 3050 1300
-Wire Wire Line
-	3050 1300 2600 1300
-Connection ~ 3300 1300
-Wire Wire Line
-	3300 1300 3050 1300
+Connection ~ 2400 1000
+Wire Wire Line
+	4500 1450 4500 1400
 Wire Wire Line
 	4800 1400 4800 1450
@@
 Wire Wire Line
 	5300 1400 5400 1400
-Connection ~ 3950 1300
-Wire Wire Line
-	3500 1300 3300 1300
-Connection ~ 3500 1300
-Wire Wire Line
-	3950 1300 3500 1300
-Wire Wire Line
-	4500 1300 3950 1300
-Wire Wire Line
-	3950 1000 4600 1000
-Connection ~ 3950 1000
-Connection ~ 3500 1000
-Wire Wire Line
-	3500 1000 3950 1000
-Wire Wire Line
-	3050 1000 3500 1000
 $Comp
 L Device:C C511
@@
 L power:+3.3V #PWR0503
 U 1 1 5A80EA7D
-P 1700 1150
+P 1150 1200
 AR Path="/5A78E64E/5A80EA7D" Ref="#PWR0503"  Part="1"
 AR Path="/5A78E661/5A80EA7D" Ref="#PWR0703"  Part="1"
-F 0 "#PWR0503" H 1700 1000 50  0001 C CNN
-F 1 "+3.3V" H 1715 1323 50  0000 C CNN
-F 2 "" H 1700 1150 50  0001 C CNN
-F 3 "" H 1700 1150 50  0001 C CNN
-	1    1700 1150
+F 0 "#PWR0503" H 1150 1050 50  0001 C CNN
+F 1 "+3.3V" H 1165 1373 50  0000 C CNN
+F 2 "" H 1150 1200 50  0001 C CNN
+F 3 "" H 1150 1200 50  0001 C CNN
+	1    1150 1200
 	1    0    0    -1
 $EndComp
@@
 L power:PWR_FLAG #FLG0501
 U 1 1 5A8B20A8
-P 2600 1000
+P 2400 1000
 AR Path="/5A78E64E/5A8B20A8" Ref="#FLG0501"  Part="1"
 AR Path="/5A78E661/5A8B20A8" Ref="#FLG0701"  Part="1"
-F 0 "#FLG0501" H 2600 1075 50  0001 C CNN
-F 1 "PWR_FLAG" H 2600 1174 50  0000 C CNN
-F 2 "" H 2600 1000 50  0001 C CNN
-F 3 "" H 2600 1000 50  0001 C CNN
-	1    2600 1000
+F 0 "#FLG0501" H 2400 1075 50  0001 C CNN
+F 1 "PWR_FLAG" H 2400 1174 50  0000 C CNN
+F 2 "" H 2400 1000 50  0001 C CNN
+F 3 "" H 2400 1000 50  0001 C CNN
+	1    2400 1000
 	1    0    0    -1
 $EndComp
@@
 L Device:L_Core_Iron L501
 U 1 1 5A852718
-P 2150 1000
+P 1600 1000
 AR Path="/5A78E64E/5A852718" Ref="L501"  Part="1"
 AR Path="/5A78E661/5A852718" Ref="L701"  Part="1"
-F 0 "L501" V 1972 1000 50  0000 C CNN
-F 1 "4u7H" V 2063 1000 50  0000 C CNN
-F 2 "Resistor_SMD:R_1210_3225Metric" H 2150 1000 50  0001 C CNN
-F 3 "https://www.murata.com/~/media/webrenewal/products/inductor/chip/tokoproducts/wirewoundmetalalloychiptype/m_dfe322512c.ashx" H 2150 1000 50  0001 C CNN
-F 4 "1277AS-H-4R7M=P2" H 2150 1000 50  0001 C CNN "mpn"
-	1    2150 1000
+F 0 "L501" V 1422 1000 50  0000 C CNN
+F 1 "4u7H" V 1513 1000 50  0000 C CNN
+F 2 "Resistor_SMD:R_1210_3225Metric" H 1600 1000 50  0001 C CNN
+F 3 "https://www.murata.com/~/media/webrenewal/products/inductor/chip/tokoproducts/wirewoundmetalalloychiptype/m_dfe322512c.ashx" H 1600 1000 50  0001 C CNN
+F 4 "1277AS-H-4R7M=P2" H 1600 1000 50  0001 C CNN "mpn"
+	1    1600 1000
 	0    1    1    0
 $EndComp
+Wire Wire Line
+	2400 1700 2400 1350
+Wire Wire Line
+	2400 1700 2050 1700
+Wire Wire Line
+	2050 1700 2050 1850
+Wire Wire Line
+	1750 1400 2050 1400
+Wire Wire Line
+	2400 1000 4600 1000
+Wire Wire Line
+	2500 1400 4500 1400
+Wire Wire Line
+	2050 1400 2500 1400
+Connection ~ 2050 1400
+Connection ~ 1900 1000
+Wire Wire Line
+	1900 1000 2400 1000
+Connection ~ 2050 1700
+Wire Wire Line
+	2050 1700 1900 1700
+Connection ~ 2500 1400
+Wire Wire Line
+	2400 1700 2500 1700
+Connection ~ 2400 1700
+Wire Wire Line
+	1900 1350 1900 1700
+Wire Wire Line
+	1900 1050 1900 1000
+Wire Wire Line
+	2400 1050 2400 1000
 $EndSCHEMATC
