File: design/Input.sch (KiCad schematic (older format))
At the start: 38 parts, among them J501 Conn_01x03, U501 93C46B, U502 FT4232H, U503 74LV595, X501 ASEMB-12MHz

Commit message: Updating capacitors for 56pin
Parts:
- removed C509, C515: 0u1F, Capacitor_SMD:C_0603_1608Metric, symbol Device:C
Connections:
- net labels added: OSCI, REF
- wire segments 186 -> 177
Changed lines of the file:
@@
 AR Path="/5A78E64E/5A7760FD" Ref="#PWR0502"  Part="1"
 AR Path="/5A78E661/5A7760FD" Ref="#PWR0702"  Part="1"
-F 0 "#PWR0502" H 1400 4650 50  0001 C CNN
+F 0 "#PWR0702" H 1400 4650 50  0001 C CNN
 F 1 "GND" H 1405 4727 50  0000 C CNN
 F 2 "" H 1400 4900 50  0001 C CNN
@@
 AR Path="/5A78E64E/5A77612B" Ref="#PWR0511"  Part="1"
 AR Path="/5A78E661/5A77612B" Ref="#PWR0711"  Part="1"
-F 0 "#PWR0511" H 4400 5750 50  0001 C CNN
+F 0 "#PWR0711" H 4400 5750 50  0001 C CNN
 F 1 "GND" H 4405 5827 50  0000 C CNN
 F 2 "" H 4400 6000 50  0001 C CNN
@@
 AR Path="/5A78E64E/5A78FA4C" Ref="#PWR0504"  Part="1"
 AR Path="/5A78E661/5A78FA4C" Ref="#PWR0704"  Part="1"
-F 0 "#PWR0504" H 2850 3200 50  0001 C CNN
+F 0 "#PWR0704" H 2850 3200 50  0001 C CNN
 F 1 "GND" H 2855 3277 50  0000 C CNN
 F 2 "" H 2850 3450 50  0001 C CNN
@@
 AR Path="/5A78E64E/5A79780B" Ref="#PWR0510"  Part="1"
 AR Path="/5A78E661/5A79780B" Ref="#PWR0710"  Part="1"
-F 0 "#PWR0510" H 3350 2150 50  0001 C CNN
+F 0 "#PWR0710" H 3350 2150 50  0001 C CNN
 F 1 "GND" H 3355 2227 50  0000 C CNN
 F 2 "" H 3350 2400 50  0001 C CNN
@@
 AR Path="/5A78E64E/5A7A5A9C" Ref="#PWR0508"  Part="1"
 AR Path="/5A78E661/5A7A5A9C" Ref="#PWR0708"  Part="1"
-F 0 "#PWR0508" H 2050 1600 50  0001 C CNN
+F 0 "#PWR0708" H 2050 1600 50  0001 C CNN
 F 1 "GND" H 2055 1677 50  0000 C CNN
 F 2 "" H 2050 1850 50  0001 C CNN
@@
 $EndComp
 $Comp
-L Device:C C509
-U 1 1 5A7D613F
-P 6050 1150
-AR Path="/5A78E64E/5A7D613F" Ref="C509"  Part="1"
-AR Path="/5A78E661/5A7D613F" Ref="C709"  Part="1"
-F 0 "C509" H 6165 1196 50  0000 L CNN
-F 1 "0u1F" H 6165 1105 50  0000 L CNN
-F 2 "Capacitor_SMD:C_0603_1608Metric" H 6088 1000 50  0001 C CNN
-F 3 "http://www.samsungsem.com/kr/support/product-search/mlcc/CL10B104KO8WPNC.jsp" H 6050 1150 50  0001 C CNN
-F 4 "CL10B104KO8WPNC" H 6050 1150 50  0001 C CNN "mpn"
-	1    6050 1150
-	1    0    0    -1
-$EndComp
-$Comp
 L Device:C C510
 U 1 1 5A7D6146
@@
 $EndComp
 $Comp
-L Device:C C515
-U 1 1 5A7DCA6C
-P 8750 1150
-AR Path="/5A78E64E/5A7DCA6C" Ref="C515"  Part="1"
-AR Path="/5A78E661/5A7DCA6C" Ref="C715"  Part="1"
-F 0 "C515" H 8865 1196 50  0000 L CNN
-F 1 "0u1F" H 8865 1105 50  0000 L CNN
-F 2 "Capacitor_SMD:C_0603_1608Metric" H 8788 1000 50  0001 C CNN
-F 3 "http://www.samsungsem.com/kr/support/product-search/mlcc/CL10B104KO8WPNC.jsp" H 8750 1150 50  0001 C CNN
-F 4 "CL10B104KO8WPNC" H 8750 1150 50  0001 C CNN "mpn"
-	1    8750 1150
-	1    0    0    -1
-$EndComp
-$Comp
 L Device:C C513
 U 1 1 5A7DCA73
@@
 AR Path="/5A78E64E/5A7DFDD9" Ref="#PWR0517"  Part="1"
 AR Path="/5A78E661/5A7DFDD9" Ref="#PWR0717"  Part="1"
-F 0 "#PWR0517" H 7400 1250 50  0001 C CNN
+F 0 "#PWR0717" H 7400 1250 50  0001 C CNN
 F 1 "GND" H 7405 1327 50  0000 C CNN
 F 2 "" H 7400 1500 50  0001 C CNN
@@
 $EndComp
 Wire Wire Line
-	6750 950  6750 850
-Connection ~ 6750 950
+	6950 950  6950 850
 Wire Wire Line
 	7400 1000 7400 950
 Wire Wire Line
-	6750 950  6950 950
-Wire Wire Line
-	6050 950  6050 1000
-Wire Wire Line
-	6050 950  6500 950
-Wire Wire Line
 	6500 1000 6500 950
-Connection ~ 6500 950
-Wire Wire Line
-	6500 950  6750 950
 Wire Wire Line
 	6950 1000 6950 950
@@
 	6950 950  7400 950
 Wire Wire Line
-	6050 1300 6050 1350
-Wire Wire Line
-	6050 1350 6500 1350
-Wire Wire Line
 	7400 1350 7400 1500
 Wire Wire Line
@@
 Wire Wire Line
 	6500 1300 6500 1350
-Connection ~ 6500 1350
 Wire Wire Line
 	6500 1350 6950 1350
@@
 	7400 1350 7850 1350
 Wire Wire Line
-	8750 1350 8750 1300
-Wire Wire Line
 	8300 1300 8300 1350
-Connection ~ 8300 1350
-Wire Wire Line
-	8300 1350 8750 1350
 Wire Wire Line
 	7850 1300 7850 1350
@@
 	7850 950  8300 950
 Wire Wire Line
-	8750 950  8750 1000
-Wire Wire Line
 	8300 1000 8300 950
 Connection ~ 8300 950
-Wire Wire Line
-	8300 950  8750 950
 NoConn ~ 6200 1950
 NoConn ~ 6200 2050
@@
 AR Path="/5A78E64E/5A808AF8" Ref="#PWR0506"  Part="1"
 AR Path="/5A78E661/5A808AF8" Ref="#PWR0706"  Part="1"
-F 0 "#PWR0506" H 3050 1550 50  0001 C CNN
+F 0 "#PWR0706" H 3050 1550 50  0001 C CNN
 F 1 "+3.3V" H 3065 1873 50  0000 C CNN
 F 2 "" H 3050 1700 50  0001 C CNN
@@
 AR Path="/5A78E64E/5A80E9F1" Ref="#PWR0512"  Part="1"
 AR Path="/5A78E661/5A80E9F1" Ref="#PWR0712"  Part="1"
-F 0 "#PWR0512" H 5300 1150 50  0001 C CNN
+F 0 "#PWR0712" H 5300 1150 50  0001 C CNN
 F 1 "+3.3V" H 5315 1473 50  0000 C CNN
 F 2 "" H 5300 1300 50  0001 C CNN
@@
 AR Path="/5A78E64E/5A80EA7D" Ref="#PWR0503"  Part="1"
 AR Path="/5A78E661/5A80EA7D" Ref="#PWR0703"  Part="1"
-F 0 "#PWR0503" H 1150 1050 50  0001 C CNN
+F 0 "#PWR0703" H 1150 1050 50  0001 C CNN
 F 1 "+3.3V" H 1165 1373 50  0000 C CNN
 F 2 "" H 1150 1200 50  0001 C CNN
@@
 L power:+3.3V #PWR0513
 U 1 1 5A814AA2
-P 6750 850
+P 6950 850
 AR Path="/5A78E64E/5A814AA2" Ref="#PWR0513"  Part="1"
 AR Path="/5A78E661/5A814AA2" Ref="#PWR0713"  Part="1"
-F 0 "#PWR0513" H 6750 700 50  0001 C CNN
-F 1 "+3.3V" H 6765 1023 50  0000 C CNN
-F 2 "" H 6750 850 50  0001 C CNN
-F 3 "" H 6750 850 50  0001 C CNN
-	1    6750 850
+F 0 "#PWR0713" H 6950 700 50  0001 C CNN
+F 1 "+3.3V" H 6965 1023 50  0000 C CNN
+F 2 "" H 6950 850 50  0001 C CNN
+F 3 "" H 6950 850 50  0001 C CNN
+	1    6950 850
 	1    0    0    -1
 $EndComp
@@
 AR Path="/5A78E64E/5A81AD3D" Ref="#PWR0516"  Part="1"
 AR Path="/5A78E661/5A81AD3D" Ref="#PWR0716"  Part="1"
-F 0 "#PWR0516" H 6900 4600 50  0001 C CNN
+F 0 "#PWR0716" H 6900 4600 50  0001 C CNN
 F 1 "+3.3V" H 6915 4923 50  0000 C CNN
 F 2 "" H 6900 4750 50  0001 C CNN
@@
 AR Path="/5A78E64E/5A820A99" Ref="#PWR0515"  Part="1"
 AR Path="/5A78E661/5A820A99" Ref="#PWR0715"  Part="1"
-F 0 "#PWR0515" H 6900 3700 50  0001 C CNN
+F 0 "#PWR0715" H 6900 3700 50  0001 C CNN
 F 1 "+3.3V" H 6915 4023 50  0000 C CNN
 F 2 "" H 6900 3850 50  0001 C CNN
@@
 AR Path="/5A78E64E/5A8267F5" Ref="#PWR0514"  Part="1"
 AR Path="/5A78E661/5A8267F5" Ref="#PWR0714"  Part="1"
-F 0 "#PWR0514" H 6900 2800 50  0001 C CNN
+F 0 "#PWR0714" H 6900 2800 50  0001 C CNN
 F 1 "+3.3V" H 6915 3123 50  0000 C CNN
 F 2 "" H 6900 2950 50  0001 C CNN
@@
 AR Path="/5A78E64E/5A8409AC" Ref="#PWR0507"  Part="1"
 AR Path="/5A78E661/5A8409AC" Ref="#PWR0707"  Part="1"
-F 0 "#PWR0507" H 3200 3600 50  0001 C CNN
+F 0 "#PWR0707" H 3200 3600 50  0001 C CNN
 F 1 "+3.3V" H 3215 3923 50  0000 C CNN
 F 2 "" H 3200 3750 50  0001 C CNN
@@
 AR Path="/5A78E64E/5A846AEB" Ref="#PWR0501"  Part="1"
 AR Path="/5A78E661/5A846AEB" Ref="#PWR0701"  Part="1"
-F 0 "#PWR0501" H 1350 4200 50  0001 C CNN
+F 0 "#PWR0701" H 1350 4200 50  0001 C CNN
 F 1 "+5V" H 1365 4523 50  0000 C CNN
 F 2 "" H 1350 4350 50  0001 C CNN
@@
 AR Path="/5A78E64E/5A848044" Ref="#PWR0509"  Part="1"
 AR Path="/5A78E661/5A848044" Ref="#PWR0709"  Part="1"
-F 0 "#PWR0509" H 3300 3100 50  0001 C CNN
+F 0 "#PWR0709" H 3300 3100 50  0001 C CNN
 F 1 "+3.3V" H 3315 3423 50  0000 C CNN
 F 2 "" H 3300 3250 50  0001 C CNN
@@
 AR Path="/5A78E64E/5A8B20A8" Ref="#FLG0501"  Part="1"
 AR Path="/5A78E661/5A8B20A8" Ref="#FLG0701"  Part="1"
-F 0 "#FLG0501" H 2400 1075 50  0001 C CNN
+F 0 "#FLG0701" H 2400 1075 50  0001 C CNN
 F 1 "PWR_FLAG" H 2400 1174 50  0000 C CNN
 F 2 "" H 2400 1000 50  0001 C CNN
@@
 AR Path="/5A78E64E/5A83C347" Ref="#PWR0521"  Part="1"
 AR Path="/5A78E661/5A83C347" Ref="#PWR0721"  Part="1"
-F 0 "#PWR0521" H 10850 4250 50  0001 C CNN
+F 0 "#PWR0721" H 10850 4250 50  0001 C CNN
 F 1 "GND" H 10855 4327 50  0000 C CNN
 F 2 "" H 10850 4500 50  0001 C CNN
@@
 AR Path="/5A78E64E/5A878935" Ref="#PWR0519"  Part="1"
 AR Path="/5A78E661/5A878935" Ref="#PWR0719"  Part="1"
-F 0 "#PWR0519" H 8850 2850 50  0001 C CNN
+F 0 "#PWR0719" H 8850 2850 50  0001 C CNN
 F 1 "+3.3V" H 8865 3173 50  0000 C CNN
 F 2 "" H 8850 3000 50  0001 C CNN
@@
 AR Path="/5A78E64E/5A878991" Ref="#PWR0520"  Part="1"
 AR Path="/5A78E661/5A878991" Ref="#PWR0720"  Part="1"
-F 0 "#PWR0520" H 8850 4250 50  0001 C CNN
+F 0 "#PWR0720" H 8850 4250 50  0001 C CNN
 F 1 "GND" H 8855 4327 50  0000 C CNN
 F 2 "" H 8850 4500 50  0001 C CNN
@@
 AR Path="/5A78E64E/5A89E551" Ref="#PWR0518"  Part="1"
 AR Path="/5A78E661/5A89E551" Ref="#PWR0718"  Part="1"
-F 0 "#PWR0518" H 7850 3300 50  0001 C CNN
+F 0 "#PWR0718" H 7850 3300 50  0001 C CNN
 F 1 "+3.3V" H 7865 3623 50  0000 C CNN
 F 2 "" H 7850 3450 50  0001 C CNN
@@
 AR Path="/5A78E64E/5A92C971" Ref="#PWR01"  Part="1"
 AR Path="/5A78E661/5A92C971" Ref="#PWR04"  Part="1"
-F 0 "#PWR01" H 2000 5300 50  0001 C CNN
+F 0 "#PWR04" H 2000 5300 50  0001 C CNN
 F 1 "GND" H 2005 5377 50  0000 C CNN
 F 2 "" H 2000 5550 50  0001 C CNN
@@
 AR Path="/5A78E64E/5A92C9CE" Ref="#PWR02"  Part="1"
 AR Path="/5A78E661/5A92C9CE" Ref="#PWR05"  Part="1"
-F 0 "#PWR02" H 2800 5600 50  0001 C CNN
+F 0 "#PWR05" H 2800 5600 50  0001 C CNN
 F 1 "GND" H 2805 5677 50  0000 C CNN
 F 2 "" H 2800 5850 50  0001 C CNN
@@
 AR Path="/5A78E64E/5A949389" Ref="#PWR03"  Part="1"
 AR Path="/5A78E661/5A949389" Ref="#PWR06"  Part="1"
-F 0 "#PWR03" H 2800 4950 50  0001 C CNN
+F 0 "#PWR06" H 2800 4950 50  0001 C CNN
 F 1 "+3.3V" H 2815 5273 50  0000 C CNN
 F 2 "" H 2800 5100 50  0001 C CNN
@@
 Wire Wire Line
 	2400 1050 2400 1000
+Text Label 3400 5500 0    50   ~ 0
+OSCI
+Text Label 3000 2950 0    50   ~ 0
+REF
+Wire Wire Line
+	6500 950  6950 950
 $EndSCHEMATC

Commit message: Renumber and sub clock generator
Parts:
- renumbered C503 to C501, C516 to C502, C501 to C503, C508 to C504, C506 to C505, C504 to C506, C510 to C508, C511 to C509, C512 to C510, C513 to C511, C514 to C512, R513 to R501, R501 to R502, R502 to R503, R503 to R504, R504 to R505, R505 to R506, R506 to R507, R507 to R508, R508 to R509, R509 to R510, R510 to R511, R511 to R512, R512 to R513

Commit message: Finish FC1 layout
Connections:
- wire segments 177 -> 176
- no-connect marks 26 -> 28
Changed lines of the file:
@@
 L Device:R_Pack08 RN501
 U 1 1 5A81550F
-P 9750 3700
+P 9750 3600
 AR Path="/5A78E64E/5A81550F" Ref="RN501"  Part="1"
 AR Path="/5A78E661/5A81550F" Ref="RN701"  Part="1"
-F 0 "RN501" V 9133 3700 50  0000 C CNN
-F 1 "330R" V 9224 3700 50  0000 C CNN
-F 2 "ResistorArray:R_Array_Convex_8x0402" V 10225 3700 50  0001 C CNN
-F 3 "https://industrial.panasonic.com/cdbs/www-data/pdf/AOC0000/AOC0000C14.pdf" H 9750 3700 50  0001 C CNN
-F 4 "EXB-2HV331JV" H 9750 3700 50  0001 C CNN "mpn"
-	1    9750 3700
-	0    1    1    0
-$EndComp
-Wire Wire Line
-	9350 3300 9550 3300
+F 0 "RN501" V 9133 3600 50  0000 C CNN
+F 1 "330R" V 9224 3600 50  0000 C CNN
+F 2 "ResistorArray:R_Array_Convex_8x0402" V 10225 3600 50  0001 C CNN
+F 3 "https://industrial.panasonic.com/cdbs/www-data/pdf/AOC0000/AOC0000C14.pdf" H 9750 3600 50  0001 C CNN
+F 4 "EXB-2HV331JV" H 9750 3600 50  0001 C CNN "mpn"
+	1    9750 3600
+	0    1    -1   0
+$EndComp
 Wire Wire Line
 	9350 3400 9550 3400
@@
 Wire Wire Line
 	6500 950  6950 950
+NoConn ~ 9550 3300
+NoConn ~ 9350 3300
 $EndSCHEMATC
