File: design/ExtComms.sch (KiCad schematic (older format))
At the start: 17 parts

Commit message: Adding Drivers for RS422 and high power LOS
Parts:
- removed R?: 1k, symbol Device:R_Small
- removed U?: FSA3157L6X, Package_SON:Fairchild_MicroPak-6_1.0x1.45mm_P0.5mm, symbol Analog_Switch:FSA3157L6X
- added C? (x2): 10uF, Resistor_SMD:R_0805_2012Metric, symbol Device:C_Small
- added C?: 0u22F, Capacitor_SMD:C_0603_1608Metric, symbol Device:C_Small
- added C? (x2): 0u1F, Capacitors_SMD:C_0603, symbol Device:C_Small
- added J?: Conn_Coaxial, symbol Connector_Specialized:Conn_Coaxial
- added J?: Conn_01x02, Connector_Phoenix_MC:PhoenixContact_MC_1,5_2-G-5.08_1x02_P5.08mm_Horizontal, symbol Connector_Generic:Conn_01x02
- added Q? (x2): Q_NMOS_DGS, Package_TO_SOT_SMD:SOT-23, symbol Device:Q_NMOS_GSD
- added R? (x2): 0R, Resistor_SMD:R_1206_3216Metric, symbol Device:R_Small
- added R?: 50R, Resistor_SMD:R_2010_5025Metric, symbol Device:R_Small
- added R? (x2): 10k, Resistors_SMD:R_0603, symbol Device:R_Small
- added R?: 120R, Resistors_SMD:R_0603, symbol Device:R_Small
- JP?: footprint (none) -> Connector_PinHeader_2.54mm:PinHeader_1x03_P2.54mm_Vertical; symbol Device:Jumper_NO_Small -> Jumper:Jumper_3_Open; mpn (none) -> M20-9990345
- U?: value MAX4427 -> TPS28225DRBT; footprint Housings_SOIC:SO-8_5.3x6.2mm_Pitch1.27mm -> Package_SON:Texas_S-PVSON-N8; symbol CommsCard:MAX4427 -> CommsCard:TPS28225
Connections:
- net labels added: +5V, GNDS, LOS_EN, LOS_OUT, PHASE, RS422_EN
- net labels removed: RS422_ENABLE
- wire segments 66 -> 104
- no-connect marks 1 -> 2
Other:
- note added: "This section can drive 5V over 50Ohm.\nEnsure all traces/components rated to 0.5W"
- moved on the sheet: U?

Commit message: Finished ERC
Parts:
- gave numbers to parts that had none: 27
Connections:
- wire segments 104 -> 103
- no-connect marks 2 -> 20
Other:
- note added: "Connect a jumper between GND and pin 1 or pin 3\nto selectively disable either LOS or RS422 transmission"
- note added: "RS232 Section"
- moved on the sheet: U302

Commit message: Swapping FT4232 for VQFN and finalizing mpns
Parts:
- J301, J302, J303: footprint Connector_Dsub:DSUB-9_Female_Horizontal_P2.77x2.84mm_EdgePinOffset7.70mm_Housed_MountingHolesOffset9.12mm -> Connector_Dsub:DSUB-9_Male_Horizontal_P2.77x2.84mm_EdgePinOffset7.70mm_Housed_MountingHolesOffset9.12mm; mpn (none) -> A-DF 09 A/KG-T2S
- J305: footprint (none) -> Connector_Coaxial:SMA_Molex_73251-1153_EdgeMount_Horizontal; mpn (none) -> 0732512120
- Q301, Q302: mpn (none) -> DMN2056U-7
- R304, R305: footprint Resistor_SMD:R_1206_3216Metric -> Resistor_SMD:R_1210_3225Metric; mpn (none) -> RMCF1210ZT0R00
- U302: footprint (none) -> Package_SO:SOIC-8_3.9x4.9mm_P1.27mm; mpn (none) -> MAX3485AEASA+
- U303: mpn (none) -> TPS28225DRBT
Changed lines of the file:
@@
 F 0 "J301" H 4279 1603 50  0000 L CNN
 F 1 "DB9_Male_MountingHoles" H 4279 1512 50  0000 L CNN
-F 2 "Connector_Dsub:DSUB-9_Female_Horizontal_P2.77x2.84mm_EdgePinOffset7.70mm_Housed_MountingHolesOffset9.12mm" H 4100 1600 50  0001 C CNN
-F 3 "" H 4100 1600 50  0001 C CNN
+F 2 "Connector_Dsub:DSUB-9_Male_Horizontal_P2.77x2.84mm_EdgePinOffset7.70mm_Housed_MountingHolesOffset9.12mm" H 4100 1600 50  0001 C CNN
+F 3 "http://www.assmann-wsw.com/fileadmin/datasheets/ASS_4888_CO.pdf" H 4100 1600 50  0001 C CNN
+F 4 "A-DF 09 A/KG-T2S" H 4100 1600 50  0001 C CNN "mpn"
 	1    4100 1600
-	1    0    0    -1
-$EndComp
-$Comp
-L Connector_Specialized:DB9_Male_MountingHoles J302
-U 1 1 5A91ED41
-P 4100 2900
-F 0 "J302" H 4279 2903 50  0000 L CNN
-F 1 "DB9_Male_MountingHoles" H 4279 2812 50  0000 L CNN
-F 2 "Connector_Dsub:DSUB-9_Female_Horizontal_P2.77x2.84mm_EdgePinOffset7.70mm_Housed_MountingHolesOffset9.12mm" H 4100 2900 50  0001 C CNN
-F 3 "" H 4100 2900 50  0001 C CNN
-	1    4100 2900
-	1    0    0    -1
-$EndComp
-$Comp
-L Connector_Specialized:DB9_Male_MountingHoles J303
-U 1 1 5A91EDCB
-P 4100 4100
-F 0 "J303" H 4279 4103 50  0000 L CNN
-F 1 "DB9_Male_MountingHoles" H 4279 4012 50  0000 L CNN
-F 2 "Connector_Dsub:DSUB-9_Female_Horizontal_P2.77x2.84mm_EdgePinOffset7.70mm_Housed_MountingHolesOffset9.12mm" H 4100 4100 50  0001 C CNN
-F 3 "" H 4100 4100 50  0001 C CNN
-	1    4100 4100
 	1    0    0    -1
 $EndComp
@@
 F 2 "Package_SON:Texas_S-PVSON-N8" H 8700 4150 50  0001 C CNN
 F 3 "http://www.ti.com/lit/ds/symlink/tps28225.pdf" H 8700 4150 50  0001 C CNN
+F 4 "TPS28225DRBT" H 0   0   50  0001 C CNN "mpn"
 	1    7900 5150
 	1    0    0    -1
@@
 F 0 "U302" H 8050 3550 50  0000 C CNN
 F 1 "MAX3485" H 8150 3450 50  0000 C CNN
-F 2 "" H 7900 2250 50  0001 C CNN
+F 2 "Package_SO:SOIC-8_3.9x4.9mm_P1.27mm" H 7900 2250 50  0001 C CNN
 F 3 "https://datasheets.maximintegrated.com/en/ds/MAX3483-MAX3491.pdf" H 7900 3000 50  0001 C CNN
+F 4 "MAX3485AEASA+" H 7900 2950 50  0001 C CNN "mpn"
 	1    7900 2950
 	1    0    0    -1
@@
 F 0 "J305" H 10499 5126 50  0000 L CNN
 F 1 "Conn_Coaxial" H 10499 5035 50  0000 L CNN
-F 2 "" H 10400 5150 50  0001 C CNN
-F 3 "" H 10400 5150 50  0001 C CNN
+F 2 "Connector_Coaxial:SMA_Molex_73251-1153_EdgeMount_Horizontal" H 10400 5150 50  0001 C CNN
+F 3 "http://www.molex.com/pdm_docs/sd/732512120_sd.pdf" H 10400 5150 50  0001 C CNN
+F 4 "0732512120" H 10400 5150 50  0001 C CNN "mpn"
 	1    10400 5150
 	1    0    0    -1
@@
 F 2 "Package_TO_SOT_SMD:SOT-23" H 9500 4800 50  0001 C CNN
 F 3 "https://www.diodes.com/assets/Datasheets/DMN2056U.pdf" H 9300 4700 50  0001 C CNN
+F 4 "DMN2056U-7" H 0   0   50  0001 C CNN "mpn"
 	1    9300 4700
 	1    0    0    -1
@@
 F 2 "Package_TO_SOT_SMD:SOT-23" H 9500 5800 50  0001 C CNN
 F 3 "https://www.diodes.com/assets/Datasheets/DMN2056U.pdf" H 9300 5700 50  0001 C CNN
+F 4 "DMN2056U-7" H 0   0   50  0001 C CNN "mpn"
 	1    9300 5700
 	1    0    0    -1
@@
 	9400 5150 9400 5500
 Connection ~ 9400 5150
-$Comp
-L Device:R_Small R305
-U 1 1 5A805C94
-P 9000 5500
-F 0 "R305" H 9059 5546 50  0000 L CNN
-F 1 "0R" H 9059 5455 50  0000 L CNN
-F 2 "Resistor_SMD:R_1206_3216Metric" H 9000 5500 50  0001 C CNN
-F 3 "~" H 9000 5500 50  0001 C CNN
-F 4 "~" H 9000 5500 50  0001 C CNN "mpn"
-	1    9000 5500
-	1    0    0    -1
-$EndComp
 Wire Wire Line
 	8350 5000 9000 5000
@@
 F 0 "R304" H 9059 4946 50  0000 L CNN
 F 1 "0R" H 9059 4855 50  0000 L CNN
-F 2 "Resistor_SMD:R_1206_3216Metric" H 9000 4900 50  0001 C CNN
-F 3 "~" H 9000 4900 50  0001 C CNN
-F 4 "~" H 9000 4900 50  0001 C CNN "mpn"
+F 2 "Resistor_SMD:R_1210_3225Metric" H 9000 4900 50  0001 C CNN
+F 3 "https://www.seielect.com/Catalog/SEI-RMCF_RMCP.pdf" H 9000 4900 50  0001 C CNN
+F 4 "RMCF1210ZT0R00" H 9000 4900 50  0001 C CNN "mpn"
 	1    9000 4900
 	1    0    0    -1
@@
 	-1   0    0    -1
 $EndComp
+$Comp
+L Connector_Specialized:DB9_Male_MountingHoles J302
+U 1 1 5A88CCB2
+P 4100 2900
+F 0 "J302" H 4279 2903 50  0000 L CNN
+F 1 "DB9_Male_MountingHoles" H 4279 2812 50  0000 L CNN
+F 2 "Connector_Dsub:DSUB-9_Male_Horizontal_P2.77x2.84mm_EdgePinOffset7.70mm_Housed_MountingHolesOffset9.12mm" H 4100 2900 50  0001 C CNN
+F 3 "http://www.assmann-wsw.com/fileadmin/datasheets/ASS_4888_CO.pdf" H 4100 2900 50  0001 C CNN
+F 4 "A-DF 09 A/KG-T2S" H 4100 2900 50  0001 C CNN "mpn"
+	1    4100 2900
+	1    0    0    -1
+$EndComp
+$Comp
+L Connector_Specialized:DB9_Male_MountingHoles J303
+U 1 1 5A88CD12
+P 4100 4100
+F 0 "J303" H 4279 4103 50  0000 L CNN
+F 1 "DB9_Male_MountingHoles" H 4279 4012 50  0000 L CNN
+F 2 "Connector_Dsub:DSUB-9_Male_Horizontal_P2.77x2.84mm_EdgePinOffset7.70mm_Housed_MountingHolesOffset9.12mm" H 4100 4100 50  0001 C CNN
+F 3 "http://www.assmann-wsw.com/fileadmin/datasheets/ASS_4888_CO.pdf" H 4100 4100 50  0001 C CNN
+F 4 "A-DF 09 A/KG-T2S" H 4100 4100 50  0001 C CNN "mpn"
+	1    4100 4100
+	1    0    0    -1
+$EndComp
+$Comp
+L Device:R_Small R305
+U 1 1 5A88D71F
+P 9000 5500
+F 0 "R305" H 9059 5546 50  0000 L CNN
+F 1 "0R" H 9059 5455 50  0000 L CNN
+F 2 "Resistor_SMD:R_1210_3225Metric" H 9000 5500 50  0001 C CNN
+F 3 "https://www.seielect.com/Catalog/SEI-RMCF_RMCP.pdf" H 9000 5500 50  0001 C CNN
+F 4 "RMCF1210ZT0R00" H 9000 5500 50  0001 C CNN "mpn"
+	1    9000 5500
+	1    0    0    -1
+$EndComp
 $EndSCHEMATC

Commit message: Updating schematic for layout
Parts:
- C301, C302, C303, C304, C305, C307, C308: footprint Capacitors_SMD:C_0603 -> Capacitor_SMD:C_0603_1608Metric; mpn CL10F104ZB8NNNC -> CL10B104KO8WPNC
- C309, C310: footprint Resistor_SMD:R_0805_2012Metric -> Capacitor_SMD:C_0805_2012Metric; mpn LMK212AB7106MG-T -> EMK212BB7106MG-T
- R301, R302: footprint Resistors_SMD:R_0603 -> Resistor_SMD:R_0603_1608Metric; mpn CRG0603F1K0 -> CRG0603J10K
- R303: footprint Resistors_SMD:R_0603 -> Resistor_SMD:R_0603_1608Metric
Changed lines of the file:
@@
 F 0 "C304" H 4115 6446 50  0000 L CNN
 F 1 "0u1F" H 4115 6355 50  0000 L CNN
-F 2 "Capacitors_SMD:C_0603" H 4038 6250 50  0001 C CNN
-F 3 "http://www.samsungsem.com/kr/support/product-search/mlcc/CL10F104ZB8NNNC.jsp" H 4000 6400 50  0001 C CNN
-F 4 "CL10F104ZB8NNNC" H 4000 6400 50  0001 C CNN "mpn"
+F 2 "Capacitor_SMD:C_0603_1608Metric" H 4038 6250 50  0001 C CNN
+F 3 "http://www.samsungsem.com/kr/support/product-search/mlcc/CL10B104KO8WPNC.jsp" H 4000 6400 50  0001 C CNN
+F 4 "CL10B104KO8WPNC" H 4000 6400 50  0001 C CNN "mpn"
 	1    4000 6400
 	-1   0    0    -1
@@
 F 0 "C305" H 4315 6446 50  0000 L CNN
 F 1 "0u1F" H 4315 6355 50  0000 L CNN
-F 2 "Capacitors_SMD:C_0603" H 4238 6250 50  0001 C CNN
-F 3 "http://www.samsungsem.com/kr/support/product-search/mlcc/CL10F104ZB8NNNC.jsp" H 4200 6400 50  0001 C CNN
-F 4 "CL10F104ZB8NNNC" H 4200 6400 50  0001 C CNN "mpn"
+F 2 "Capacitor_SMD:C_0603_1608Metric" H 4238 6250 50  0001 C CNN
+F 3 "http://www.samsungsem.com/kr/support/product-search/mlcc/CL10B104KO8WPNC.jsp" H 4200 6400 50  0001 C CNN
+F 4 "CL10B104KO8WPNC" H 4200 6400 50  0001 C CNN "mpn"
 	1    4200 6400
 	1    0    0    -1
@@
 F 0 "C303" H 2565 6546 50  0000 L CNN
 F 1 "0u1F" H 2565 6455 50  0000 L CNN
-F 2 "Capacitors_SMD:C_0603" H 2488 6350 50  0001 C CNN
-F 3 "http://www.samsungsem.com/kr/support/product-search/mlcc/CL10F104ZB8NNNC.jsp" H 2450 6500 50  0001 C CNN
-F 4 "CL10F104ZB8NNNC" H 2450 6500 50  0001 C CNN "mpn"
+F 2 "Capacitor_SMD:C_0603_1608Metric" H 2488 6350 50  0001 C CNN
+F 3 "http://www.samsungsem.com/kr/support/product-search/mlcc/CL10B104KO8WPNC.jsp" H 2450 6500 50  0001 C CNN
+F 4 "CL10B104KO8WPNC" H 2450 6500 50  0001 C CNN "mpn"
 	1    2450 6500
 	-1   0    0    -1
@@
 F 0 "C302" H 2565 6046 50  0000 L CNN
 F 1 "0u1F" H 2565 5955 50  0000 L CNN
-F 2 "Capacitors_SMD:C_0603" H 2488 5850 50  0001 C CNN
-F 3 "http://www.samsungsem.com/kr/support/product-search/mlcc/CL10F104ZB8NNNC.jsp" H 2450 6000 50  0001 C CNN
-F 4 "CL10F104ZB8NNNC" H 2450 6000 50  0001 C CNN "mpn"
+F 2 "Capacitor_SMD:C_0603_1608Metric" H 2488 5850 50  0001 C CNN
+F 3 "http://www.samsungsem.com/kr/support/product-search/mlcc/CL10B104KO8WPNC.jsp" H 2450 6000 50  0001 C CNN
+F 4 "CL10B104KO8WPNC" H 2450 6000 50  0001 C CNN "mpn"
 	1    2450 6000
 	-1   0    0    -1
@@
 F 0 "C301" H 2065 5796 50  0000 L CNN
 F 1 "0u1F" H 2065 5705 50  0000 L CNN
-F 2 "Capacitors_SMD:C_0603" H 1988 5600 50  0001 C CNN
-F 3 "http://www.samsungsem.com/kr/support/product-search/mlcc/CL10F104ZB8NNNC.jsp" H 1950 5750 50  0001 C CNN
-F 4 "CL10F104ZB8NNNC" H 1950 5750 50  0001 C CNN "mpn"
+F 2 "Capacitor_SMD:C_0603_1608Metric" H 1988 5600 50  0001 C CNN
+F 3 "http://www.samsungsem.com/kr/support/product-search/mlcc/CL10B104KO8WPNC.jsp" H 1950 5750 50  0001 C CNN
+F 4 "CL10B104KO8WPNC" H 1950 5750 50  0001 C CNN "mpn"
 	1    1950 5750
 	-1   0    0    -1
@@
 F 0 "R302" H 8130 1004 50  0000 R CNN
 F 1 "10k" H 8130 1095 50  0000 R CNN
-F 2 "Resistors_SMD:R_0603" V 8130 1050 50  0001 C CNN
+F 2 "Resistor_SMD:R_0603_1608Metric" V 8130 1050 50  0001 C CNN
 F 3 "http://www.te.com/commerce/DocumentDelivery/DDEController?Action=srchrtrv&DocNm=1773204&DocType=DS&DocLang=English" H 8200 1050 50  0001 C CNN
-F 4 "CRG0603F1K0" H 8200 1050 50  0001 C CNN "mpn"
+F 4 "CRG0603J10K" H 8200 1050 50  0001 C CNN "mpn"
 	1    8200 1050
 	-1   0    0    1
@@
 F 0 "R301" H 7530 1004 50  0000 R CNN
 F 1 "10k" H 7530 1095 50  0000 R CNN
-F 2 "Resistors_SMD:R_0603" V 7530 1050 50  0001 C CNN
+F 2 "Resistor_SMD:R_0603_1608Metric" V 7530 1050 50  0001 C CNN
 F 3 "http://www.te.com/commerce/DocumentDelivery/DDEController?Action=srchrtrv&DocNm=1773204&DocType=DS&DocLang=English" H 7600 1050 50  0001 C CNN
-F 4 "CRG0603F1K0" H 7600 1050 50  0001 C CNN "mpn"
+F 4 "CRG0603J10K" H 7600 1050 50  0001 C CNN "mpn"
 	1    7600 1050
 	1    0    0    1
@@
 F 0 "C309" V 10121 4450 50  0000 C CNN
 F 1 "10uF" V 10212 4450 50  0000 C CNN
-F 2 "Resistor_SMD:R_0805_2012Metric" H 10350 4450 50  0001 C CNN
+F 2 "Capacitor_SMD:C_0805_2012Metric" H 10350 4450 50  0001 C CNN
 F 3 "https://www.yuden.co.jp/productdata/catalog/mlcc_all_e.pdf" H 10350 4450 50  0001 C CNN
-F 4 "LMK212AB7106MG-T" H 10350 4450 50  0001 C CNN "mpn"
+F 4 "EMK212BB7106MG-T" H 10350 4450 50  0001 C CNN "mpn"
 	1    10350 4450
 	1    0    0    1
@@
 F 0 "C310" V 10421 4450 50  0000 C CNN
 F 1 "10uF" V 10512 4450 50  0000 C CNN
-F 2 "Resistor_SMD:R_0805_2012Metric" H 10650 4450 50  0001 C CNN
+F 2 "Capacitor_SMD:C_0805_2012Metric" H 10650 4450 50  0001 C CNN
 F 3 "https://www.yuden.co.jp/productdata/catalog/mlcc_all_e.pdf" H 10650 4450 50  0001 C CNN
-F 4 "LMK212AB7106MG-T" H 10650 4450 50  0001 C CNN "mpn"
+F 4 "EMK212BB7106MG-T" H 10650 4450 50  0001 C CNN "mpn"
 	1    10650 4450
 	-1   0    0    1
@@
 F 0 "C308" H 7665 4396 50  0000 L CNN
 F 1 "0u1F" H 7665 4305 50  0000 L CNN
-F 2 "Capacitors_SMD:C_0603" H 7588 4200 50  0001 C CNN
-F 3 "http://www.samsungsem.com/kr/support/product-search/mlcc/CL10F104ZB8NNNC.jsp" H 7550 4350 50  0001 C CNN
-F 4 "CL10F104ZB8NNNC" H 7550 4350 50  0001 C CNN "mpn"
+F 2 "Capacitor_SMD:C_0603_1608Metric" H 7588 4200 50  0001 C CNN
+F 3 "http://www.samsungsem.com/kr/support/product-search/mlcc/CL10B104KO8WPNC.jsp" H 7550 4350 50  0001 C CNN
+F 4 "CL10B104KO8WPNC" H 7550 4350 50  0001 C CNN "mpn"
 	1    7550 4350
 	1    0    0    -1
@@
 F 0 "C307" H 7415 2396 50  0000 L CNN
 F 1 "0u1F" H 7415 2305 50  0000 L CNN
-F 2 "Capacitors_SMD:C_0603" H 7338 2200 50  0001 C CNN
-F 3 "http://www.samsungsem.com/kr/support/product-search/mlcc/CL10F104ZB8NNNC.jsp" H 7300 2350 50  0001 C CNN
-F 4 "CL10F104ZB8NNNC" H 7300 2350 50  0001 C CNN "mpn"
+F 2 "Capacitor_SMD:C_0603_1608Metric" H 7338 2200 50  0001 C CNN
+F 3 "http://www.samsungsem.com/kr/support/product-search/mlcc/CL10B104KO8WPNC.jsp" H 7300 2350 50  0001 C CNN
+F 4 "CL10B104KO8WPNC" H 7300 2350 50  0001 C CNN "mpn"
 	1    7300 2350
 	-1   0    0    -1
@@
 F 0 "R303" H 8530 2954 50  0000 R CNN
 F 1 "120R" H 8530 3045 50  0000 R CNN
-F 2 "Resistors_SMD:R_0603" V 8530 3000 50  0001 C CNN
+F 2 "Resistor_SMD:R_0603_1608Metric" V 8530 3000 50  0001 C CNN
 F 3 "http://www.yageo.com/documents/recent/PYu-RT_1-to-0.01_RoHS_L_9.pdf" H 8600 3000 50  0001 C CNN
 F 4 "RT0603DRE07120RL" H 8600 3000 50  0001 C CNN "mpn"
