File: design/Watchdog.sch (KiCad schematic (older format))
At the start: 0 parts

Commit message: Adding watchdog
Parts:
- added U? (x2): STWD100xxWY, symbol CommsCard:STWD100xxWY
Changed lines of the file:
@@
 $Descr A4 11693 8268
 encoding utf-8
-Sheet 1 7
+Sheet 5 7
 Title ""
 Date ""
@@
 Comment4 ""
 $EndDescr
+$Comp
+L CommsCard:STWD100xxWY U?
+U 1 1 5A7B0FE8
+P 5900 4050
+F 0 "U?" H 6291 4096 50  0000 L CNN
+F 1 "STWD100xxWY" H 6291 4005 50  0000 L CNN
+F 2 "" H 5950 4250 50  0001 C CNN
+F 3 "http://www.st.com/content/ccc/resource/technical/document/datasheet/06/6a/b3/83/9a/c7/4f/22/CD00176077.pdf/files/CD00176077.pdf/jcr:content/translations/en.CD00176077.pdf" H 6050 4350 50  0001 C CNN
+	1    5900 4050
+	1    0    0    -1
+$EndComp
+$Comp
+L CommsCard:STWD100xxWY U?
+U 1 1 5A7B1006
+P 5850 2700
+F 0 "U?" H 6241 2746 50  0000 L CNN
+F 1 "STWD100xxWY" H 6241 2655 50  0000 L CNN
+F 2 "" H 5900 2900 50  0001 C CNN
+F 3 "http://www.st.com/content/ccc/resource/technical/document/datasheet/06/6a/b3/83/9a/c7/4f/22/CD00176077.pdf/files/CD00176077.pdf/jcr:content/translations/en.CD00176077.pdf" H 6000 3000 50  0001 C CNN
+	1    5850 2700
+	1    0    0    -1
+$EndComp
 $EndSCHEMATC

Commit message: Adding TI footprint and watchdog stuff
Parts:
- added R? (x3): R, symbol Device:R
- added TP? (x2): Test_Point, symbol Connector_Specialized:Test_Point
- added U? (x2): 74LVC2G00, Package_BGA:Texas_DSBGA-8_0.9x1.9mm_Layout2x4_P0.5mm, symbol CommsCard:74LVC2G00
- added U?: 74AHC157, symbol CommsCard:74AHC157RGY
Connections:
- net labels added: +3V3, FC1_PWREN, FC1_WD, FC2_PWREN, FC2_WD, GND
- wire segments 0 -> 33

Commit message: Updating wd
Parts:
- removed TP?: Test_Point, symbol Connector_Specialized:Test_Point
- removed U?: STWD100xxWY, symbol CommsCard:STWD100xxWY
- added C? (x4): 0u1F, Capacitor_SMD:C_0603_1608Metric, symbol Device:C
- added TP?: Test_Point, Measurement_Points:Measurement_Point_Round-SMD-Pad_Small, symbol Connector_Specialized:Test_Point
- added U?: 74LVC2G00, Package_BGA:Texas_DSBGA-8_0.9x1.9mm_Layout2x4_P0.5mm, symbol CommsCard:74LVC2G00
- added U?: STWD100xxWY, TO_SOT_Packages_SMD:SOT-353_SC-70-5, symbol CommsCard:STWD100xxWY
- R? (x2): footprint (none) -> Resistors_SMD:R_0603
- TP?: footprint (none) -> Measurement_Points:Measurement_Point_Round-SMD-Pad_Small
- U?: footprint (none) -> TO_SOT_Packages_SMD:SOT-353_SC-70-5; mpn (none) -> STWD100PYW83F
Connections:
- wire segments 33 -> 52
Changed lines of the file:
@@
 F 0 "U?" H 5191 4296 50  0000 L CNN
 F 1 "STWD100xxWY" H 5191 4205 50  0000 L CNN
-F 2 "" H 4850 4450 50  0001 C CNN
+F 2 "TO_SOT_Packages_SMD:SOT-353_SC-70-5" H 4850 4450 50  0001 C CNN
 F 3 "http://www.st.com/content/ccc/resource/technical/document/datasheet/06/6a/b3/83/9a/c7/4f/22/CD00176077.pdf/files/CD00176077.pdf/jcr:content/translations/en.CD00176077.pdf" H 4950 4550 50  0001 C CNN
+F 4 "STWD100PYW83F" H 4800 4250 50  0001 C CNN "mpn"
 	1    4800 4250
-	1    0    0    -1
-$EndComp
-$Comp
-L CommsCard:STWD100xxWY U?
-U 1 1 5A7B1006
-P 4750 2850
-F 0 "U?" H 5141 2896 50  0000 L CNN
-F 1 "STWD100xxWY" H 5141 2805 50  0000 L CNN
-F 2 "" H 4800 3050 50  0001 C CNN
-F 3 "http://www.st.com/content/ccc/resource/technical/document/datasheet/06/6a/b3/83/9a/c7/4f/22/CD00176077.pdf/files/CD00176077.pdf/jcr:content/translations/en.CD00176077.pdf" H 4900 3150 50  0001 C CNN
-	1    4750 2850
 	1    0    0    -1
 $EndComp
@@
 F 0 "TP?" H 4208 2620 50  0000 L CNN
 F 1 "Test_Point" H 4208 2529 50  0000 L CNN
-F 2 "" H 4350 2500 50  0001 C CNN
+F 2 "Measurement_Points:Measurement_Point_Round-SMD-Pad_Small" H 4350 2500 50  0001 C CNN
 F 3 "~" H 4350 2500 50  0001 C CNN
 	1    4150 2500
@@
 F 0 "R?" H 3380 4104 50  0000 R CNN
 F 1 "R" H 3380 4195 50  0000 R CNN
-F 2 "" V 3380 4150 50  0001 C CNN
+F 2 "Resistors_SMD:R_0603" V 3380 4150 50  0001 C CNN
 F 3 "~" H 3450 4150 50  0001 C CNN
+F 4 "~" H 3450 4150 50  0001 C CNN "mpn"
 	1    3450 4150
 	-1   0    0    1
@@
 F 0 "R?" H 3330 2704 50  0000 R CNN
 F 1 "R" H 3330 2795 50  0000 R CNN
-F 2 "" V 3330 2750 50  0001 C CNN
+F 2 "Resistors_SMD:R_0603" V 3330 2750 50  0001 C CNN
 F 3 "~" H 3400 2750 50  0001 C CNN
 	1    3400 2750
@@
 Text HLabel 3400 2950 0    50   Input ~ 0
 FC1_PWREN
-$Comp
-L Connector_Specialized:Test_Point TP?
-U 1 1 5A7B9083
-P 4200 3900
-F 0 "TP?" H 4258 4020 50  0000 L CNN
-F 1 "Test_Point" H 4258 3929 50  0000 L CNN
-F 2 "" H 4400 3900 50  0001 C CNN
-F 3 "~" H 4400 3900 50  0001 C CNN
-	1    4200 3900
-	1    0    0    -1
-$EndComp
 $Comp
 L power:+3V3 #PWR?
@@
 	9200 4050 9200 4000
 Connection ~ 9100 4050
+$Comp
+L CommsCard:74LVC2G00 U?
+U 3 1 5A7BD6BD
+P 5800 5650
+F 0 "U?" H 5775 5917 50  0000 C CNN
+F 1 "74LVC2G00" H 5775 5826 50  0000 C CNN
+F 2 "Package_BGA:Texas_DSBGA-8_0.9x1.9mm_Layout2x4_P0.5mm" H 5800 5650 50  0001 C CNN
+F 3 "http://www.ti.com/lit/ds/symlink/sn74lvc2g00.pdf" H 5800 5650 50  0001 C CNN
+F 4 "SN74LVC2G00YZPR" H 5800 5650 50  0001 C CNN "mpn"
+	3    5800 5650
+	1    0    0    -1
+$EndComp
+$Comp
+L power:+3V3 #PWR?
+U 1 1 5A7BD74A
+P 5800 5050
+F 0 "#PWR?" H 5800 4900 50  0001 C CNN
+F 1 "+3V3" H 5815 5223 50  0000 C CNN
+F 2 "" H 5800 5050 50  0001 C CNN
+F 3 "" H 5800 5050 50  0001 C CNN
+	1    5800 5050
+	1    0    0    -1
+$EndComp
+$Comp
+L power:GND #PWR?
+U 1 1 5A7BD781
+P 5800 6250
+F 0 "#PWR?" H 5800 6000 50  0001 C CNN
+F 1 "GND" H 5805 6077 50  0000 C CNN
+F 2 "" H 5800 6250 50  0001 C CNN
+F 3 "" H 5800 6250 50  0001 C CNN
+	1    5800 6250
+	1    0    0    -1
+$EndComp
+$Comp
+L CommsCard:STWD100xxWY U?
+U 1 1 5A7BE12B
+P 4750 2850
+F 0 "U?" H 5141 2896 50  0000 L CNN
+F 1 "STWD100xxWY" H 5141 2805 50  0000 L CNN
+F 2 "TO_SOT_Packages_SMD:SOT-353_SC-70-5" H 4800 3050 50  0001 C CNN
+F 3 "http://www.st.com/content/ccc/resource/technical/document/datasheet/06/6a/b3/83/9a/c7/4f/22/CD00176077.pdf/files/CD00176077.pdf/jcr:content/translations/en.CD00176077.pdf" H 4900 3150 50  0001 C CNN
+F 4 "STWD100PYW83F" H 4750 2850 50  0001 C CNN "mpn"
+	1    4750 2850
+	1    0    0    -1
+$EndComp
+$Comp
+L Connector_Specialized:Test_Point TP?
+U 1 1 5A7BE190
+P 4200 3900
+F 0 "TP?" H 4258 4020 50  0000 L CNN
+F 1 "Test_Point" H 4258 3929 50  0000 L CNN
+F 2 "Measurement_Points:Measurement_Point_Round-SMD-Pad_Small" H 4400 3900 50  0001 C CNN
+F 3 "~" H 4400 3900 50  0001 C CNN
+	1    4200 3900
+	1    0    0    -1
+$EndComp
+Wire Wire Line
+	6200 5500 6200 5050
+Wire Wire Line
+	6200 5800 6200 6200
+$Comp
+L Device:C C?
+U 1 1 5A7C0E16
+P 6200 5650
+F 0 "C?" H 6315 5696 50  0000 L CNN
+F 1 "0u1F" H 6315 5605 50  0000 L CNN
+F 2 "Capacitor_SMD:C_0603_1608Metric" H 6238 5500 50  0001 C CNN
+F 3 "~" H 6200 5650 50  0001 C CNN
+F 4 "CL10B104KA8NFNC" H 6200 5650 50  0001 C CNN "mpn"
+	1    6200 5650
+	1    0    0    -1
+$EndComp
+Wire Wire Line
+	6650 5500 6650 5050
+Wire Wire Line
+	6650 5800 6650 6200
+$Comp
+L Device:C C?
+U 1 1 5A7C13BB
+P 6650 5650
+F 0 "C?" H 6765 5696 50  0000 L CNN
+F 1 "0u1F" H 6765 5605 50  0000 L CNN
+F 2 "Capacitor_SMD:C_0603_1608Metric" H 6688 5500 50  0001 C CNN
+F 3 "~" H 6650 5650 50  0001 C CNN
+F 4 "CL10B104KA8NFNC" H 6650 5650 50  0001 C CNN "mpn"
+	1    6650 5650
+	1    0    0    -1
+$EndComp
+Wire Wire Line
+	7100 5500 7100 5050
+Wire Wire Line
+	7100 5800 7100 6200
+$Comp
+L Device:C C?
+U 1 1 5A7C1A22
+P 7100 5650
+F 0 "C?" H 7215 5696 50  0000 L CNN
+F 1 "0u1F" H 7215 5605 50  0000 L CNN
+F 2 "Capacitor_SMD:C_0603_1608Metric" H 7138 5500 50  0001 C CNN
+F 3 "~" H 7100 5650 50  0001 C CNN
+F 4 "CL10B104KA8NFNC" H 7100 5650 50  0001 C CNN "mpn"
+	1    7100 5650
+	1    0    0    -1
+$EndComp
+Wire Wire Line
+	7550 5500 7550 5050
+Wire Wire Line
+	7550 5800 7550 6200
+$Comp
+L Device:C C?
+U 1 1 5A7C1A2B
+P 7550 5650
+F 0 "C?" H 7665 5696 50  0000 L CNN
+F 1 "0u1F" H 7665 5605 50  0000 L CNN
+F 2 "Capacitor_SMD:C_0603_1608Metric" H 7588 5500 50  0001 C CNN
+F 3 "~" H 7550 5650 50  0001 C CNN
+F 4 "CL10B104KA8NFNC" H 7550 5650 50  0001 C CNN "mpn"
+	1    7550 5650
+	1    0    0    -1
+$EndComp
+Wire Wire Line
+	5800 6250 5800 6200
+Wire Wire Line
+	5800 6200 6200 6200
+Connection ~ 5800 6200
+Wire Wire Line
+	5800 6200 5800 6000
+Connection ~ 6200 6200
+Wire Wire Line
+	6200 6200 6650 6200
+Connection ~ 6650 6200
+Wire Wire Line
+	6650 6200 7100 6200
+Connection ~ 7100 6200
+Wire Wire Line
+	7100 6200 7550 6200
+Wire Wire Line
+	5800 5300 5800 5050
+Wire Wire Line
+	5800 5050 6200 5050
+Connection ~ 5800 5050
+Connection ~ 6200 5050
+Wire Wire Line
+	6200 5050 6650 5050
+Connection ~ 6650 5050
+Wire Wire Line
+	6650 5050 7100 5050
+Connection ~ 7100 5050
+Wire Wire Line
+	7100 5050 7550 5050
 $EndSCHEMATC

Commit message: Connecting LOS inside FC connection
Connections:
- net labels added: COMM1_TX, COMM2_TX, FC1_COMM1_TX, FC1_COMM2_TX, FC1_HIGHRATE, FC1_LOS, FC2_COMM1_TX, FC2_COMM2_TX, FC2_HIGHRATE, FC2_LOS, HIGHRATE, IN_CHARGE, LOS, ~FC1_PWREN, ~FC2_PWREN
- net labels removed: FC1_PWREN, FC2_PWREN
- wire segments 52 -> 56
Changed lines of the file:
@@
 $Descr A4 11693 8268
 encoding utf-8
-Sheet 5 7
+Sheet 4 8
 Title ""
 Date ""
@@
 	3450 4000 3450 3950
 Text HLabel 3450 4350 0    50   Input ~ 0
-FC2_PWREN
+~FC2_PWREN
 Wire Wire Line
 	3400 2950 3400 2900
@@
 	3400 2600 3400 2550
 Text HLabel 3400 2950 0    50   Input ~ 0
-FC1_PWREN
+~FC1_PWREN
 $Comp
 L power:+3V3 #PWR?
@@
 Wire Wire Line
 	7100 5050 7550 5050
+Text HLabel 8600 2400 0    50   Input ~ 0
+FC1_COMM1_TX
+Text HLabel 8600 2500 0    50   Input ~ 0
+FC2_COMM1_TX
+Text HLabel 8600 2800 0    50   Input ~ 0
+FC2_COMM2_TX
+Text HLabel 8600 2700 0    50   Input ~ 0
+FC1_COMM2_TX
+Text HLabel 8600 3000 0    50   Input ~ 0
+FC1_HIGHRATE
+Text HLabel 8600 3100 0    50   Input ~ 0
+FC2_HIGHRATE
+Text HLabel 8600 3300 0    50   Input ~ 0
+FC1_LOS
+Text HLabel 8600 3400 0    50   Input ~ 0
+FC2_LOS
+Text HLabel 9600 2400 2    50   Output ~ 0
+COMM1_TX
+Text HLabel 9600 2700 2    50   Output ~ 0
+COMM2_TX
+Text HLabel 9600 3000 2    50   Output ~ 0
+HIGHRATE
+Text HLabel 9600 3300 2    50   Output ~ 0
+LOS
+Wire Wire Line
+	8600 3700 8600 4050
+Wire Wire Line
+	8600 4050 9000 4050
+Connection ~ 9000 4050
+Wire Wire Line
+	7400 3600 7400 4000
+Wire Wire Line
+	7400 4000 7650 4000
+Text HLabel 7650 4000 2    50   Output ~ 0
+IN_CHARGE
 $EndSCHEMATC

Commit message: Finished ERC
Parts:
- gave numbers to parts that had none: 14
Changed lines of the file:
@@
 $Descr A4 11693 8268
 encoding utf-8
-Sheet 4 8
+Sheet 4 10
 Title ""
 Date ""
@@
 $EndDescr
 $Comp
-L CommsCard:STWD100xxWY U?
+L CommsCard:STWD100xxWY U402
 U 1 1 5A7B0FE8
 P 4800 4250
-F 0 "U?" H 5191 4296 50  0000 L CNN
+F 0 "U402" H 5191 4296 50  0000 L CNN
 F 1 "STWD100xxWY" H 5191 4205 50  0000 L CNN
 F 2 "TO_SOT_Packages_SMD:SOT-353_SC-70-5" H 4850 4450 50  0001 C CNN
@@
 $EndComp
 $Comp
-L CommsCard:74LVC2G00 U?
+L CommsCard:74LVC2G00 U404
 U 2 1 5A7B6676
 P 6700 4200
-F 0 "U?" H 6675 4467 50  0000 C CNN
+F 0 "U404" H 6675 4467 50  0000 C CNN
 F 1 "74LVC2G00" H 6675 4376 50  0000 C CNN
 F 2 "Package_BGA:Texas_DSBGA-8_0.9x1.9mm_Layout2x4_P0.5mm" H 6700 4200 50  0001 C CNN
@@
 	6200 2950 6400 2950
 $Comp
-L Device:R R?
+L Device:R R403
 U 1 1 5A7B69B9
 P 7150 2900
-F 0 "R?" V 6943 2900 50  0000 C CNN
+F 0 "R403" V 6943 2900 50  0000 C CNN
 F 1 "R" V 7034 2900 50  0000 C CNN
 F 2 "" V 7080 2900 50  0001 C CNN
@@
 	6400 2850 5100 2850
 $Comp
-L power:GND #PWR?
+L power:GND #PWR0404
 U 1 1 5A7B7021
 P 4750 3250
-F 0 "#PWR?" H 4750 3000 50  0001 C CNN
+F 0 "#PWR0404" H 4750 3000 50  0001 C CNN
 F 1 "GND" H 4755 3077 50  0000 C CNN
 F 2 "" H 4750 3250 50  0001 C CNN
@@
 	4750 3250 4750 3200
 $Comp
-L power:GND #PWR?
+L power:GND #PWR0406
 U 1 1 5A7B7145
 P 4800 4650
-F 0 "#PWR?" H 4800 4400 50  0001 C CNN
+F 0 "#PWR0406" H 4800 4400 50  0001 C CNN
 F 1 "GND" H 4805 4477 50  0000 C CNN
 F 2 "" H 4800 4650 50  0001 C CNN
@@
 	4800 4650 4800 4600
 $Comp
-L CommsCard:74LVC2G00 U?
+L CommsCard:74LVC2G00 U403
 U 2 1 5A7B74F5
 P 6700 2900
-F 0 "U?" H 6675 3167 50  0000 C CNN
+F 0 "U403" H 6675 3167 50  0000 C CNN
 F 1 "74LVC2G00" H 6675 3076 50  0000 C CNN
 F 2 "Package_BGA:Texas_DSBGA-8_0.9x1.9mm_Layout2x4_P0.5mm" H 6700 2900 50  0001 C CNN
@@
 FC1_WD
 $Comp
-L Connector_Specialized:Test_Point TP?
+L Connector_Specialized:Test_Point TP401
 U 1 1 5A7B77EA
 P 4150 2500
-F 0 "TP?" H 4208 2620 50  0000 L CNN
+F 0 "TP401" H 4208 2620 50  0000 L CNN
 F 1 "Test_Point" H 4208 2529 50  0000 L CNN
 F 2 "Measurement_Points:Measurement_Point_Round-SMD-Pad_Small" H 4350 2500 50  0001 C CNN
@@
 	3450 4350 4450 4350
 $Comp
-L power:+3V3 #PWR?
+L power:+3V3 #PWR0402
 U 1 1 5A7B80F0
 P 3450 3950
-F 0 "#PWR?" H 3450 3800 50  0001 C CNN
+F 0 "#PWR0402" H 3450 3800 50  0001 C CNN
 F 1 "+3V3" H 3465 4123 50  0000 C CNN
 F 2 "" H 3450 3950 50  0001 C CNN
@@
 $EndComp
 $Comp
-L Device:R R?
+L Device:R R402
 U 1 1 5A7B810E
 P 3450 4150
-F 0 "R?" H 3380 4104 50  0000 R CNN
+F 0 "R402" H 3380 4104 50  0000 R CNN
 F 1 "R" H 3380 4195 50  0000 R CNN
 F 2 "Resistors_SMD:R_0603" V 3380 4150 50  0001 C CNN
@@
 	3400 2950 4400 2950
 $Comp
-L power:+3V3 #PWR?
+L power:+3V3 #PWR0401
 U 1 1 5A7B889A
 P 3400 2550
-F 0 "#PWR?" H 3400 2400 50  0001 C CNN
+F 0 "#PWR0401" H 3400 2400 50  0001 C CNN
 F 1 "+3V3" H 3415 2723 50  0000 C CNN
 F 2 "" H 3400 2550 50  0001 C CNN
@@
 $EndComp
 $Comp
-L Device:R R?
+L Device:R R401
 U 1 1 5A7B88A0
 P 3400 2750
-F 0 "R?" H 3330 2704 50  0000 R CNN
+F 0 "R401" H 3330 2704 50  0000 R CNN
 F 1 "R" H 3330 2795 50  0000 R CNN
 F 2 "Resistors_SMD:R_0603" V 3330 2750 50  0001 C CNN
@@
 ~FC1_PWREN
 $Comp
-L power:+3V3 #PWR?
+L power:+3V3 #PWR0405
 U 1 1 5A7B9113
 P 4800 3900
-F 0 "#PWR?" H 4800 3750 50  0001 C CNN
+F 0 "#PWR0405" H 4800 3750 50  0001 C CNN
 F 1 "+3V3" H 4815 4073 50  0000 C CNN
 F 2 "" H 4800 3900 50  0001 C CNN
@@
 $EndComp
 $Comp
-L power:+3V3 #PWR?
+L power:+3V3 #PWR0403
 U 1 1 5A7B9130
 P 4750 2500
-F 0 "#PWR?" H 4750 2350 50  0001 C CNN
+F 0 "#PWR0403" H 4750 2350 50  0001 C CNN
 F 1 "+3V3" H 4765 2673 50  0000 C CNN
 F 2 "" H 4750 2500 50  0001 C CNN
@@
 $EndComp
 $Comp
-L CommsCard:74AHC157RGY U?
+L CommsCard:74AHC157RGY U405
 U 1 1 5A7BA9FB
 P 9100 3000
-F 0 "U?" H 9200 3900 50  0000 C CNN
+F 0 "U405" H 9200 3900 50  0000 C CNN
 F 1 "74AHC157" H 9350 3800 50  0000 C CNN
 F 2 "" H 9100 3000 50  0001 C CNN
@@
 Connection ~ 7400 3600
 $Comp
-L power:+3V3 #PWR?
+L power:+3V3 #PWR0409
 U 1 1 5A7BE16C
 P 9100 2100
-F 0 "#PWR?" H 9100 1950 50  0001 C CNN
+F 0 "#PWR0409" H 9100 1950 50  0001 C CNN
 F 1 "+3V3" H 9115 2273 50  0000 C CNN
 F 2 "" H 9100 2100 50  0001 C CNN
@@
 $EndComp
 $Comp
-L power:GND #PWR?
+L power:GND #PWR0410
 U 1 1 5A7BE18B
 P 9100 4100
-F 0 "#PWR?" H 9100 3850 50  0001 C CNN
+F 0 "#PWR0410" H 9100 3850 50  0001 C CNN
 F 1 "GND" H 9105 3927 50  0000 C CNN
 F 2 "" H 9100 4100 50  0001 C CNN
@@
 Connection ~ 9100 4050
 $Comp
-L CommsCard:74LVC2G00 U?
+L CommsCard:74LVC2G00 U403
 U 3 1 5A7BD6BD
 P 5800 5650
-F 0 "U?" H 5775 5917 50  0000 C CNN
+F 0 "U403" H 5775 5917 50  0000 C CNN
 F 1 "74LVC2G00" H 5775 5826 50  0000 C CNN
 F 2 "Package_BGA:Texas_DSBGA-8_0.9x1.9mm_Layout2x4_P0.5mm" H 5800 5650 50  0001 C CNN
@@
 $EndComp
 $Comp
-L power:+3V3 #PWR?
+L power:+3V3 #PWR0407
 U 1 1 5A7BD74A
 P 5800 5050
-F 0 "#PWR?" H 5800 4900 50  0001 C CNN
+F 0 "#PWR0407" H 5800 4900 50  0001 C CNN
 F 1 "+3V3" H 5815 5223 50  0000 C CNN
 F 2 "" H 5800 5050 50  0001 C CNN
@@
 $EndComp
 $Comp
-L power:GND #PWR?
+L power:GND #PWR0408
 U 1 1 5A7BD781
 P 5800 6250
-F 0 "#PWR?" H 5800 6000 50  0001 C CNN
+F 0 "#PWR0408" H 5800 6000 50  0001 C CNN
 F 1 "GND" H 5805 6077 50  0000 C CNN
 F 2 "" H 5800 6250 50  0001 C CNN
@@
 $EndComp
 $Comp
-L CommsCard:STWD100xxWY U?
+L CommsCard:STWD100xxWY U401
 U 1 1 5A7BE12B
 P 4750 2850
-F 0 "U?" H 5141 2896 50  0000 L CNN
+F 0 "U401" H 5141 2896 50  0000 L CNN
 F 1 "STWD100xxWY" H 5141 2805 50  0000 L CNN
 F 2 "TO_SOT_Packages_SMD:SOT-353_SC-70-5" H 4800 3050 50  0001 C CNN
@@
 $EndComp
 $Comp
-L Connector_Specialized:Test_Point TP?
+L Connector_Specialized:Test_Point TP402
 U 1 1 5A7BE190
 P 4200 3900
-F 0 "TP?" H 4258 4020 50  0000 L CNN
+F 0 "TP402" H 4258 4020 50  0000 L CNN
 F 1 "Test_Point" H 4258 3929 50  0000 L CNN
 F 2 "Measurement_Points:Measurement_Point_Round-SMD-Pad_Small" H 4400 3900 50  0001 C CNN
@@
 	6200 5800 6200 6200
 $Comp
-L Device:C C?
+L Device:C C401
 U 1 1 5A7C0E16
 P 6200 5650
-F 0 "C?" H 6315 5696 50  0000 L CNN
+F 0 "C401" H 6315 5696 50  0000 L CNN
 F 1 "0u1F" H 6315 5605 50  0000 L CNN
 F 2 "Capacitor_SMD:C_0603_1608Metric" H 6238 5500 50  0001 C CNN
@@
 	6650 5800 6650 6200
 $Comp
-L Device:C C?
+L Device:C C402
 U 1 1 5A7C13BB
 P 6650 5650
-F 0 "C?" H 6765 5696 50  0000 L CNN
+F 0 "C402" H 6765 5696 50  0000 L CNN
 F 1 "0u1F" H 6765 5605 50  0000 L CNN
 F 2 "Capacitor_SMD:C_0603_1608Metric" H 6688 5500 50  0001 C CNN
@@
 	7100 5800 7100 6200
 $Comp
-L Device:C C?
+L Device:C C403
 U 1 1 5A7C1A22
 P 7100 5650
-F 0 "C?" H 7215 5696 50  0000 L CNN
+F 0 "C403" H 7215 5696 50  0000 L CNN
 F 1 "0u1F" H 7215 5605 50  0000 L CNN
 F 2 "Capacitor_SMD:C_0603_1608Metric" H 7138 5500 50  0001 C CNN
@@
 	7550 5800 7550 6200
 $Comp
-L Device:C C?
+L Device:C C404
 U 1 1 5A7C1A2B
 P 7550 5650
-F 0 "C?" H 7665 5696 50  0000 L CNN
+F 0 "C404" H 7665 5696 50  0000 L CNN
 F 1 "0u1F" H 7665 5605 50  0000 L CNN
 F 2 "Capacitor_SMD:C_0603_1608Metric" H 7588 5500 50  0001 C CNN

Commit message: Adding more indicators
Parts:
- removed R402: R, Resistors_SMD:R_0603, symbol Device:R
- added D? (x2): Red, LED_THT:LED_D5.0mm_Horizontal_O6.35mm_Z9.0mm, symbol Device:LED_ALT
- added D?: LED_Dual_ACA, symbol Device:LED_Dual_ACA
- added R?: 10k, Resistors_SMD:R_0603, symbol Device:R
- added R? (x4): 49R9, Resistor_SMD:R_0603_1608Metric, symbol Device:R_Small
- added TP403: Test_Point, Measurement_Points:Measurement_Point_Round-SMD-Pad_Small, symbol Connector_Specialized:Test_Point
- added U? (x4): 74HC04, symbol Logic_74xx:74HC04
- R401: value R -> 10k; mpn (none) -> CRG0603F1K0
- R403: value R -> 10k; footprint (none) -> Resistors_SMD:R_0603; mpn (none) -> CRG0603F1K0
Connections:
- wire segments 56 -> 74

Commit message: Swapping FT4232 for VQFN and finalizing mpns
Parts:
- removed U? (x3): 74HC04, symbol Logic_74xx:74HC04
- added C405: 0u1F, Capacitor_SMD:C_0603_1608Metric, symbol Device:C
- added unit 4 of U406
- added unit 2 of U406
- added unit 1 of U406
- added unit 7 of U406
- D403: renamed from D?; footprint (none) -> LED_THT:LED_D8.0mm-3; mpn (none) -> WP130WDT/EYW
- U405: footprint (none) -> Package_SO:TSSOP-16_4.4x5mm_P0.65mm
- U406: renamed from U?; footprint (none) -> Package_SO:TSSOP-14_4.4x5mm_P0.65mm; mpn (none) -> SN74HC04PWR
- gave numbers to parts that had none: 7
Connections:
- wire segments 74 -> 82
Other:
- moved on the sheet: U406C

Commit message: Updating schematic for layout
Parts:
- added C406: 0u1F, Capacitor_SMD:C_0603_1608Metric, symbol Device:C
- added JP401: Jumper_NO_Small, Connector_PinHeader_2.54mm:PinHeader_1x03_P2.54mm_Vertical, symbol Jumper:Jumper_3_Open
- C401, C402, C403, C404, C405: mpn CL10B104KA8NFNC -> CL10B104KO8WPNC
- R401, R402, R403: footprint Resistors_SMD:R_0603 -> Resistor_SMD:R_0603_1608Metric; mpn CRG0603F1K0 -> CRG0603J10K
- TP401, TP402, TP403: footprint Measurement_Points:Measurement_Point_Round-SMD-Pad_Small -> TestPoint:TestPoint_Pad_D1.5mm
- U401, U402: footprint TO_SOT_Packages_SMD:SOT-353_SC-70-5 -> Package_TO_SOT_SMD:SOT-353_SC-70-5
- U403: renamed from U404; footprint Package_BGA:Texas_DSBGA-8_0.9x1.9mm_Layout2x4_P0.5mm -> Package_SO:VSSOP-8_2.3x2mm_P0.5mm; mpn SN74LVC2G00YZPR -> SN74LVC2G00DCUR
- U403: footprint Package_BGA:Texas_DSBGA-8_0.9x1.9mm_Layout2x4_P0.5mm -> Package_SO:VSSOP-8_2.3x2mm_P0.5mm; mpn SN74LVC2G00YZPR -> SN74LVC2G00DCUR
- U405: footprint Package_SO:TSSOP-16_4.4x5mm_P0.65mm -> TI-QFN:Texas_R-PVQFN-N16_EP4x3.5_Pitch0.5mm
- U406: value 74HC04 -> 74LV14; mpn SN74HC04PWR -> SN74LV14APWR
Connections:
- net labels added: +3.3V
- wire segments 82 -> 89
Other:
- note added: "Connect a jumper on pins 1-2 for FC1\nConnect a jumper on pins 2-3 for FC2\nLeave open for watchdog select"
- note added: "InCharge Override"
