File: design/LOSComms.sch (KiCad schematic (older format))
At the start: 16 parts, among them U1 SN74LV86, U2 74LV14, U3 74LVC1G80, U4 74LVC2G86, U5 74LVC2G86, U6 74LV595, U7 74LV595

Commit message: Remove annotation
Parts:
- renumbered C1 to C?, C2 to C?, C3 to C?, C4 to C?, C5 to C?, C6 to C?, C7 to C?, U4 to U?, U5 to U?, U7 to U?, U1 to U?, U2 to U?, U6 to U?, U3 to U?
Changed lines of the file:
@@
 $EndDescr
 $Comp
-L Logic_74xx:74LS595 U6
+L Logic_74xx:74LS595 U?
 U 1 1 5A7B0A9F
 P 7150 3050
-F 0 "U6" H 7300 3750 50  0000 C CNN
+F 0 "U?" H 7300 3750 50  0000 C CNN
 F 1 "74LV595" H 7400 3650 50  0000 C CNN
 F 2 "Package_SO:TSSOP-16_4.4x5mm_P0.65mm" H 7150 3050 50  0001 C CNN
@@
 	9550 3150 9450 3150
 $Comp
-L CommsCard:74LVC2G86 U4
+L CommsCard:74LVC2G86 U?
 U 1 1 5A7A4A0A
 P 6250 2650
-F 0 "U4" H 6225 2917 50  0000 C CNN
+F 0 "U?" H 6225 2917 50  0000 C CNN
 F 1 "74LVC2G86" H 6225 2826 50  0000 C CNN
 F 2 "Package_SO:MSOP-8_3x3mm_P0.65mm" H 6250 2650 50  0001 C CNN
@@
 $EndComp
 $Comp
-L power:GND #PWR01
+L power:GND #PWR?
 U 1 1 5A7A4E0B
 P 7150 3900
-F 0 "#PWR01" H 7150 3650 50  0001 C CNN
+F 0 "#PWR?" H 7150 3650 50  0001 C CNN
 F 1 "GND" H 7155 3727 50  0000 C CNN
 F 2 "" H 7150 3900 50  0001 C CNN
@@
 $EndComp
 $Comp
-L power:GND #PWR02
+L power:GND #PWR?
 U 1 1 5A7A4E27
 P 8950 3900
-F 0 "#PWR02" H 8950 3650 50  0001 C CNN
+F 0 "#PWR?" H 8950 3650 50  0001 C CNN
 F 1 "GND" H 8955 3727 50  0000 C CNN
 F 2 "" H 8950 3900 50  0001 C CNN
@@
 NoConn ~ 9450 3550
 $Comp
-L CommsCard:74LVC2G86 U4
+L CommsCard:74LVC2G86 U?
 U 2 1 5A7A5077
 P 9850 3100
-F 0 "U4" H 9825 3367 50  0000 C CNN
+F 0 "U?" H 9825 3367 50  0000 C CNN
 F 1 "74LVC2G86" H 9825 3276 50  0000 C CNN
 F 2 "Package_SO:MSOP-8_3x3mm_P0.65mm" H 9850 3100 50  0001 C CNN
@@
 $EndComp
 $Comp
-L CommsCard:74LVC2G86 U5
+L CommsCard:74LVC2G86 U?
 U 3 1 5A7A513D
 P 9350 5650
-F 0 "U5" H 9428 5696 50  0000 L CNN
+F 0 "U?" H 9428 5696 50  0000 L CNN
 F 1 "74LVC2G86" H 9428 5605 50  0000 L CNN
 F 2 "Package_SO:MSOP-8_3x3mm_P0.65mm" H 9350 5650 50  0001 C CNN
@@
 	6500 2650 6600 2650
 $Comp
-L Logic_74xx:74LS595 U7
+L Logic_74xx:74LS595 U?
 U 1 1 5A7A5871
 P 8950 3050
-F 0 "U7" H 9100 3750 50  0000 C CNN
+F 0 "U?" H 9100 3750 50  0000 C CNN
 F 1 "74LV595" H 9200 3650 50  0000 C CNN
 F 2 "Package_SO:TSSOP-16_4.4x5mm_P0.65mm" H 8950 3050 50  0001 C CNN
@@
 	7150 2350 7150 2250
 $Comp
-L power:+3V3 #PWR03
+L power:+3V3 #PWR?
 U 1 1 5A7A63A7
 P 7150 2250
-F 0 "#PWR03" H 7150 2100 50  0001 C CNN
+F 0 "#PWR?" H 7150 2100 50  0001 C CNN
 F 1 "+3V3" H 7165 2423 50  0000 C CNN
 F 2 "" H 7150 2250 50  0001 C CNN
@@
 	8950 2350 8950 2250
 $Comp
-L power:+3V3 #PWR04
+L power:+3V3 #PWR?
 U 1 1 5A7A63C9
 P 8950 2250
-F 0 "#PWR04" H 8950 2100 50  0001 C CNN
+F 0 "#PWR?" H 8950 2100 50  0001 C CNN
 F 1 "+3V3" H 8965 2423 50  0000 C CNN
 F 2 "" H 8950 2250 50  0001 C CNN
@@
 	5300 2700 5950 2700
 $Comp
-L power:+3V3 #PWR05
+L power:+3V3 #PWR?
 U 1 1 5A7A6D06
 P 5850 2950
-F 0 "#PWR05" H 5850 2800 50  0001 C CNN
+F 0 "#PWR?" H 5850 2800 50  0001 C CNN
 F 1 "+3V3" H 5865 3123 50  0000 C CNN
 F 2 "" H 5850 2950 50  0001 C CNN
@@
 $EndComp
 $Comp
-L power:+3V3 #PWR06
+L power:+3V3 #PWR?
 U 1 1 5A7A7242
 P 7850 2950
-F 0 "#PWR06" H 7850 2800 50  0001 C CNN
+F 0 "#PWR?" H 7850 2800 50  0001 C CNN
 F 1 "+3V3" H 7865 3123 50  0000 C CNN
 F 2 "" H 7850 2950 50  0001 C CNN
@@
 NoConn ~ 7650 3250
 $Comp
-L CommsCard:74LVC2G86 U4
+L CommsCard:74LVC2G86 U?
 U 3 1 5A7AD935
 P 8300 5650
-F 0 "U4" H 8378 5696 50  0000 L CNN
+F 0 "U?" H 8378 5696 50  0000 L CNN
 F 1 "74LVC2G86" H 8378 5605 50  0000 L CNN
 F 2 "Package_SO:MSOP-8_3x3mm_P0.65mm" H 8300 5650 50  0001 C CNN
@@
 $EndComp
 $Comp
-L Logic_74xx:74LS86 U1
+L Logic_74xx:74LS86 U?
 U 1 1 5A7ADAF8
 P 1550 4550
-F 0 "U1" H 1550 4875 50  0000 C CNN
+F 0 "U?" H 1550 4875 50  0000 C CNN
 F 1 "SN74LV86" H 1550 4784 50  0000 C CNN
 F 2 "Package_SO:TSSOP-14_4.4x5mm_P0.65mm" H 1550 4550 50  0001 C CNN
@@
 $EndComp
 $Comp
-L Logic_74xx:74LS86 U1
+L Logic_74xx:74LS86 U?
 U 2 1 5A7ADC31
 P 1550 5150
-F 0 "U1" H 1550 5475 50  0000 C CNN
+F 0 "U?" H 1550 5475 50  0000 C CNN
 F 1 "SN74LV86" H 1550 5384 50  0000 C CNN
 F 2 "Package_SO:TSSOP-14_4.4x5mm_P0.65mm" H 1550 5150 50  0001 C CNN
@@
 $EndComp
 $Comp
-L Logic_74xx:74LS86 U1
+L Logic_74xx:74LS86 U?
 U 3 1 5A7ADC99
 P 3150 5650
-F 0 "U1" H 3150 5975 50  0000 C CNN
+F 0 "U?" H 3150 5975 50  0000 C CNN
 F 1 "SN74LV86" H 3150 5884 50  0000 C CNN
 F 2 "Package_SO:TSSOP-14_4.4x5mm_P0.65mm" H 3150 5650 50  0001 C CNN
@@
 $EndComp
 $Comp
-L Logic_74xx:74LV14 U2
+L Logic_74xx:74LV14 U?
 U 1 1 5A7ADF20
 P 2250 5550
-F 0 "U2" H 2250 5867 50  0000 C CNN
+F 0 "U?" H 2250 5867 50  0000 C CNN
 F 1 "74LV14" H 2250 5776 50  0000 C CNN
 F 2 "Package_SO:TSSOP-14_4.4x5mm_P0.65mm" H 2250 5550 50  0001 C CNN
@@
 $EndComp
 $Comp
-L Device:C C1
+L Device:C C?
 U 1 1 5A7AE61F
 P 2650 5350
-F 0 "C1" H 2765 5396 50  0000 L CNN
+F 0 "C?" H 2765 5396 50  0000 L CNN
 F 1 "DNP" H 2765 5305 50  0000 L CNN
 F 2 "Capacitor_SMD:C_0603_1608Metric" H 2688 5200 50  0001 C CNN
@@
 	1950 5150 1850 5150
 $Comp
-L power:GND #PWR07
+L power:GND #PWR?
 U 1 1 5A7B0922
 P 1200 5350
-F 0 "#PWR07" H 1200 5100 50  0001 C CNN
+F 0 "#PWR?" H 1200 5100 50  0001 C CNN
 F 1 "GND" H 1205 5177 50  0000 C CNN
 F 2 "" H 1200 5350 50  0001 C CNN
@@
 	1100 4650 1250 4650
 $Comp
-L CommsCard:74LVC1G80 U3
+L CommsCard:74LVC1G80 U?
 U 1 1 5A7B4C81
 P 3900 4650
-F 0 "U3" H 3900 4967 50  0000 C CNN
+F 0 "U?" H 3900 4967 50  0000 C CNN
 F 1 "74LVC1G80" H 3900 4876 50  0000 C CNN
 F 2 "Package_TO_SOT_SMD:SOT-353_SC-70-5" H 3900 4650 50  0001 C CNN
@@
 	3650 4550 1850 4550
 $Comp
-L Logic_74xx:74LV14 U2
+L Logic_74xx:74LV14 U?
 U 2 1 5A7BEEBC
 P 2150 2850
-F 0 "U2" H 2150 3167 50  0000 C CNN
+F 0 "U?" H 2150 3167 50  0000 C CNN
 F 1 "74LV14" H 2150 3076 50  0000 C CNN
 F 2 "Package_SO:TSSOP-14_4.4x5mm_P0.65mm" H 2150 2850 50  0001 C CNN
@@
 	2450 2850 2750 2850
 $Comp
-L Logic_74xx:74LV14 U2
+L Logic_74xx:74LV14 U?
 U 3 1 5A7C0A07
 P 3400 2850
-F 0 "U2" H 3400 3167 50  0000 C CNN
+F 0 "U?" H 3400 3167 50  0000 C CNN
 F 1 "74LV14" H 3400 3076 50  0000 C CNN
 F 2 "Package_SO:TSSOP-14_4.4x5mm_P0.65mm" H 3400 2850 50  0001 C CNN
@@
 $EndComp
 $Comp
-L Logic_74xx:74LS86 U1
+L Logic_74xx:74LS86 U?
 U 5 1 5A7C2776
 P 4950 5700
-F 0 "U1" H 5180 5746 50  0000 L CNN
+F 0 "U?" H 5180 5746 50  0000 L CNN
 F 1 "SN74LV86" H 5180 5655 50  0000 L CNN
 F 2 "Package_SO:TSSOP-14_4.4x5mm_P0.65mm" H 4950 5700 50  0001 C CNN
@@
 $EndComp
 $Comp
-L Logic_74xx:74LV14 U2
+L Logic_74xx:74LV14 U?
 U 7 1 5A7C2856
 P 6250 5700
-F 0 "U2" H 6480 5746 50  0000 L CNN
+F 0 "U?" H 6480 5746 50  0000 L CNN
 F 1 "74LV14" H 6480 5655 50  0000 L CNN
 F 2 "Package_SO:TSSOP-14_4.4x5mm_P0.65mm" H 6250 5700 50  0001 C CNN
@@
 $EndComp
 $Comp
-L CommsCard:74LVC1G80 U3
+L CommsCard:74LVC1G80 U?
 U 2 1 5A7C605D
 P 7250 5650
-F 0 "U3" H 7330 5671 50  0000 L CNN
+F 0 "U?" H 7330 5671 50  0000 L CNN
 F 1 "74LVC1G80" H 7330 5580 50  0000 L CNN
 F 2 "Package_TO_SOT_SMD:SOT-353_SC-70-5" H 7250 5650 50  0001 C CNN
@@
 $EndComp
 $Comp
-L power:GND #PWR010
+L power:GND #PWR?
 U 1 1 5A7C9996
 P 7250 6300
-F 0 "#PWR010" H 7250 6050 50  0001 C CNN
+F 0 "#PWR?" H 7250 6050 50  0001 C CNN
 F 1 "GND" H 7255 6127 50  0000 C CNN
 F 2 "" H 7250 6300 50  0001 C CNN
@@
 Connection ~ 8300 6250
 $Comp
-L power:+3V3 #PWR09
+L power:+3V3 #PWR?
 U 1 1 5A7CE773
 P 7250 5050
-F 0 "#PWR09" H 7250 4900 50  0001 C CNN
+F 0 "#PWR?" H 7250 4900 50  0001 C CNN
 F 1 "+3V3" H 7265 5223 50  0000 C CNN
 F 2 "" H 7250 5050 50  0001 C CNN
@@
 This delay is between 2ns and 46ns over -40 to 125C.\nAdditional delay with optional capacitor
 $Comp
-L Device:C C2
+L Device:C C?
 U 1 1 5A81E8DA
 P 2750 3050
-F 0 "C2" H 2865 3096 50  0000 L CNN
+F 0 "C?" H 2865 3096 50  0000 L CNN
 F 1 "DNP" H 2865 3005 50  0000 L CNN
 F 2 "Capacitor_SMD:C_0603_1608Metric" H 2788 2900 50  0001 C CNN
@@
 $EndComp
 $Comp
-L power:GND #PWR08
+L power:GND #PWR?
 U 1 1 5A81E9A7
 P 2750 3250
-F 0 "#PWR08" H 2750 3000 50  0001 C CNN
+F 0 "#PWR?" H 2750 3000 50  0001 C CNN
 F 1 "GND" H 2755 3077 50  0000 C CNN
 F 2 "" H 2750 3250 50  0001 C CNN
@@
 	2750 3250 2750 3200
 $Comp
-L Device:C C3
+L Device:C C?
 U 1 1 5A82356F
 P 4400 5700
-F 0 "C3" H 4515 5746 50  0000 L CNN
+F 0 "C?" H 4515 5746 50  0000 L CNN
 F 1 "0u1F" H 4515 5655 50  0000 L CNN
 F 2 "Capacitor_SMD:C_0603_1608Metric" H 4438 5550 50  0001 C CNN
@@
 $EndComp
 $Comp
-L Device:C C4
+L Device:C C?
 U 1 1 5A823695
 P 5700 5700
-F 0 "C4" H 5815 5746 50  0000 L CNN
+F 0 "C?" H 5815 5746 50  0000 L CNN
 F 1 "0u1F" H 5815 5655 50  0000 L CNN
 F 2 "Capacitor_SMD:C_0603_1608Metric" H 5738 5550 50  0001 C CNN
@@
 $EndComp
 $Comp
-L Device:C C5
+L Device:C C?
 U 1 1 5A823707
 P 6850 5700
-F 0 "C5" H 6965 5746 50  0000 L CNN
+F 0 "C?" H 6965 5746 50  0000 L CNN
 F 1 "0u1F" H 6965 5655 50  0000 L CNN
 F 2 "Capacitor_SMD:C_0603_1608Metric" H 6888 5550 50  0001 C CNN
@@
 $EndComp
 $Comp
-L Device:C C6
+L Device:C C?
 U 1 1 5A823767
 P 7900 5700
-F 0 "C6" H 8015 5746 50  0000 L CNN
+F 0 "C?" H 8015 5746 50  0000 L CNN
 F 1 "0u1F" H 8015 5655 50  0000 L CNN
 F 2 "Capacitor_SMD:C_0603_1608Metric" H 7938 5550 50  0001 C CNN
@@
 $EndComp
 $Comp
-L Device:C C7
+L Device:C C?
 U 1 1 5A8237CD
 P 8950 5700
-F 0 "C7" H 9065 5746 50  0000 L CNN
+F 0 "C?" H 9065 5746 50  0000 L CNN
 F 1 "0u1F" H 9065 5655 50  0000 L CNN
 F 2 "Capacitor_SMD:C_0603_1608Metric" H 8988 5550 50  0001 C CNN

Commit message: Adding Drivers for RS422 and high power LOS
Changed lines of the file:
@@
 $Descr A4 11693 8268
 encoding utf-8
-Sheet 7 8
+Sheet 6 8
 Title ""
 Date ""
@@
 U 1 1 5A7B0A9F
 P 7150 3050
+AR Path="/5A78E64E/5A7DC371/5A7B0A9F" Ref="U?"  Part="1"
+AR Path="/5A78E661/5A7DC371/5A7B0A9F" Ref="U?"  Part="1"
 F 0 "U?" H 7300 3750 50  0000 C CNN
 F 1 "74LV595" H 7400 3650 50  0000 C CNN
@@
 U 1 1 5A7A4A0A
 P 6250 2650
+AR Path="/5A78E64E/5A7DC371/5A7A4A0A" Ref="U?"  Part="1"
+AR Path="/5A78E661/5A7DC371/5A7A4A0A" Ref="U?"  Part="1"
 F 0 "U?" H 6225 2917 50  0000 C CNN
 F 1 "74LVC2G86" H 6225 2826 50  0000 C CNN
@@
 U 2 1 5A7A5077
 P 9850 3100
+AR Path="/5A78E64E/5A7DC371/5A7A5077" Ref="U?"  Part="2"
+AR Path="/5A78E661/5A7DC371/5A7A5077" Ref="U?"  Part="2"
 F 0 "U?" H 9825 3367 50  0000 C CNN
 F 1 "74LVC2G86" H 9825 3276 50  0000 C CNN
@@
 U 3 1 5A7A513D
 P 9350 5650
+AR Path="/5A78E64E/5A7DC371/5A7A513D" Ref="U?"  Part="3"
+AR Path="/5A78E661/5A7DC371/5A7A513D" Ref="U?"  Part="3"
 F 0 "U?" H 9428 5696 50  0000 L CNN
 F 1 "74LVC2G86" H 9428 5605 50  0000 L CNN
@@
 U 1 1 5A7A5871
 P 8950 3050
+AR Path="/5A78E64E/5A7DC371/5A7A5871" Ref="U?"  Part="1"
+AR Path="/5A78E661/5A7DC371/5A7A5871" Ref="U?"  Part="1"
 F 0 "U?" H 9100 3750 50  0000 C CNN
 F 1 "74LV595" H 9200 3650 50  0000 C CNN
@@
 Wire Wire Line
 	5850 2950 6650 2950
-Wire Notes Line rgb(194, 0, 0)
+Wire Notes Line width 12 rgb(194, 0, 0)
 	10400 4550 5150 4550
-Wire Notes Line width 10 style dotted rgb(194, 0, 0)
+Wire Notes Line width 12 style dotted rgb(194, 0, 0)
 	5150 4550 5150 1950
-Wire Notes Line rgb(194, 0, 0)
+Wire Notes Line width 12 rgb(194, 0, 0)
 	5150 1950 10400 1950
-Wire Notes Line rgb(194, 0, 0)
+Wire Notes Line width 12 rgb(194, 0, 0)
 	10400 1950 10400 4550
 Text Notes 5150 1950 0    50   ~ 0
@@
 U 3 1 5A7AD935
 P 8300 5650
+AR Path="/5A78E64E/5A7DC371/5A7AD935" Ref="U?"  Part="3"
+AR Path="/5A78E661/5A7DC371/5A7AD935" Ref="U?"  Part="3"
 F 0 "U?" H 8378 5696 50  0000 L CNN
 F 1 "74LVC2G86" H 8378 5605 50  0000 L CNN
@@
 U 1 1 5A7ADAF8
 P 1550 4550
+AR Path="/5A78E64E/5A7DC371/5A7ADAF8" Ref="U?"  Part="1"
+AR Path="/5A78E661/5A7DC371/5A7ADAF8" Ref="U?"  Part="1"
 F 0 "U?" H 1550 4875 50  0000 C CNN
 F 1 "SN74LV86" H 1550 4784 50  0000 C CNN
@@
 U 2 1 5A7ADC31
 P 1550 5150
+AR Path="/5A78E64E/5A7DC371/5A7ADC31" Ref="U?"  Part="2"
+AR Path="/5A78E661/5A7DC371/5A7ADC31" Ref="U?"  Part="2"
 F 0 "U?" H 1550 5475 50  0000 C CNN
 F 1 "SN74LV86" H 1550 5384 50  0000 C CNN
@@
 U 3 1 5A7ADC99
 P 3150 5650
+AR Path="/5A78E64E/5A7DC371/5A7ADC99" Ref="U?"  Part="3"
+AR Path="/5A78E661/5A7DC371/5A7ADC99" Ref="U?"  Part="3"
 F 0 "U?" H 3150 5975 50  0000 C CNN
 F 1 "SN74LV86" H 3150 5884 50  0000 C CNN
@@
 U 1 1 5A7ADF20
 P 2250 5550
+AR Path="/5A78E64E/5A7DC371/5A7ADF20" Ref="U?"  Part="1"
+AR Path="/5A78E661/5A7DC371/5A7ADF20" Ref="U?"  Part="1"
 F 0 "U?" H 2250 5867 50  0000 C CNN
 F 1 "74LV14" H 2250 5776 50  0000 C CNN
@@
 U 1 1 5A7B4C81
 P 3900 4650
+AR Path="/5A78E64E/5A7DC371/5A7B4C81" Ref="U?"  Part="1"
+AR Path="/5A78E661/5A7DC371/5A7B4C81" Ref="U?"  Part="1"
 F 0 "U?" H 3900 4967 50  0000 C CNN
 F 1 "74LVC1G80" H 3900 4876 50  0000 C CNN
@@
 U 2 1 5A7BEEBC
 P 2150 2850
+AR Path="/5A78E64E/5A7DC371/5A7BEEBC" Ref="U?"  Part="2"
+AR Path="/5A78E661/5A7DC371/5A7BEEBC" Ref="U?"  Part="2"
 F 0 "U?" H 2150 3167 50  0000 C CNN
 F 1 "74LV14" H 2150 3076 50  0000 C CNN
@@
 U 3 1 5A7C0A07
 P 3400 2850
+AR Path="/5A78E64E/5A7DC371/5A7C0A07" Ref="U?"  Part="3"
+AR Path="/5A78E661/5A7DC371/5A7C0A07" Ref="U?"  Part="3"
 F 0 "U?" H 3400 3167 50  0000 C CNN
 F 1 "74LV14" H 3400 3076 50  0000 C CNN
@@
 U 5 1 5A7C2776
 P 4950 5700
+AR Path="/5A78E64E/5A7DC371/5A7C2776" Ref="U?"  Part="5"
+AR Path="/5A78E661/5A7DC371/5A7C2776" Ref="U?"  Part="5"
 F 0 "U?" H 5180 5746 50  0000 L CNN
 F 1 "SN74LV86" H 5180 5655 50  0000 L CNN
@@
 U 7 1 5A7C2856
 P 6250 5700
+AR Path="/5A78E64E/5A7DC371/5A7C2856" Ref="U?"  Part="7"
+AR Path="/5A78E661/5A7DC371/5A7C2856" Ref="U?"  Part="7"
 F 0 "U?" H 6480 5746 50  0000 L CNN
 F 1 "74LV14" H 6480 5655 50  0000 L CNN
@@
 U 2 1 5A7C605D
 P 7250 5650
+AR Path="/5A78E64E/5A7DC371/5A7C605D" Ref="U?"  Part="2"
+AR Path="/5A78E661/5A7DC371/5A7C605D" Ref="U?"  Part="2"
 F 0 "U?" H 7330 5671 50  0000 L CNN
 F 1 "74LVC1G80" H 7330 5580 50  0000 L CNN
@@
 Text Notes 1200 6400 0    50   ~ 0
 NOTE: Set C1 to 1nF for 70ns pulse width, 200pF for 30ns, open 10ns
-Text Notes 1650 2300 0    50   ~ 0
+Text Notes 4250 2300 2    50   ~ 0
 This delay is between 2ns and 46ns over -40 to 125C.\nAdditional delay with optional capacitor
 $Comp
@@
 Wire Wire Line
 	10050 5100 9350 5100
+Wire Notes Line width 12
+	4300 2350 4300 3550
+Wire Notes Line width 12
+	4300 3550 1350 3550
+Wire Notes Line width 12
+	1350 3550 1350 2350
+Wire Notes Line width 12
+	1350 2350 4300 2350
 $EndSCHEMATC

Commit message: Finished ERC
Parts:
- gave numbers to parts that had none: 16

Commit message: Updating schematic for layout
Parts:
- removed unit 1 of U602
- removed unit 3 of U602
- removed unit 7 of U602
- added U602 (x2): 74LVC3G14, Package_SO:VSSOP-8_2.3x2mm_P0.5mm, symbol CommsCard:74LVC3G14
- added unit 4 of U602
- C603, C604, C605, C606, C607, C608, C609: mpn CL10B104KA8NFNC -> CL10B104KO8WPNC
- U602: value 74LV14 -> 74LVC3G14; footprint Package_SO:TSSOP-14_4.4x5mm_P0.65mm -> Package_SO:VSSOP-8_2.3x2mm_P0.5mm; symbol Logic_74xx:74LV14 -> CommsCard:74LVC3G14; mpn SN74LV14APWR -> SN74LVC3G14DCUR
Other:
- note added: "Bi-Phase Signal"
- note added: "NOTE: Set C601/C801 to 1nF for 70ns pulse width, 200pF for 30ns, open 10ns"
- note added: "RNRZ-L Signal"
- note removed: "NOTE: Set C1 to 1nF for 70ns pulse width, 200pF for 30ns, open 10ns"
- note removed: "RNRZ-L"
- moved on the sheet: U804, U806

Commit message: Renumber and sub clock generator
Parts:
- removed C601: DNP, Capacitor_SMD:C_0603_1608Metric, symbol Device:C
- removed unit 2 of U601
- removed unit 3 of U601
- removed U602: 74LVC3G14, Package_SO:VSSOP-8_2.3x2mm_P0.5mm, symbol CommsCard:74LVC3G14
- removed unit 1 of U604
- removed unit 2 of U604
- added C602: 0u1F, Capacitor_SMD:C_0603_1608Metric, symbol Device:C
- added unit 2 of U602
- added unit 3 of U602
- added U603: 501BMILF, Package_SO:SOIC-8_3.9x4.9mm_P1.27mm, symbol CommsCard:501BMILF
- renumbered C602 to C601, U602 to U601, U601 to U602, U603 to U604, U604 to U606, U606 to U607, U607 to U608
Connections:
- wire segments 98 -> 97
- no-connect marks 15 -> 19
Other:
- note removed: "NOTE: Set C601/C801 to 1nF for 70ns pulse width, 200pF for 30ns, open 10ns"

Commit message: Annotating
Parts:
- removed C608, C609: 0u1F, Capacitor_SMD:C_0603_1608Metric, symbol Device:C
- removed U606, U608: 74LVC2G86, Package_SO:MSOP-8_3x3mm_P0.65mm, symbol CommsCard:74LVC2G86
- renumbered C603 to C801, C602 to C802, C605 to C803, C604 to C804, C607 to C805, C606 to C806, C601 to C807, U601 to U801, U602 to U802, U603 to U803, U604 to U804, U605 to U805, U607 to U806
Connections:
- wire segments 97 -> 83
