File: design/LOSComms.sch (KiCad schematic (older format))
At the start: 13 parts, among them U801 74LVC3G14, U802 SN74LV86, U803 501BMILF, U804 74LVC1G80, U805 74LV595, U806 74LV595

Commit message: Propogate Power nets
Parts:
- renumbered C801 to C601, C802 to C602, C803 to C603, C804 to C604, C805 to C605, C806 to C606, C807 to C607, U801 to U601, U802 to U602, U803 to U603, U804 to U604, U805 to U605, U806 to U606
Other:
- moved on the sheet: C607

Commit message: Adding labels to LOS nets
Connections:
- net labels added: 2xCLOCK, RAW_BIPHASE
Changed lines of the file:
@@
 AR Path="/5A78E64E/5A7DC371/5A7B0A9F" Ref="U605"  Part="1"
 AR Path="/5A78E661/5A7DC371/5A7B0A9F" Ref="U805"  Part="1"
-F 0 "U605" H 7900 2600 50  0000 C CNN
+F 0 "U805" H 7900 2600 50  0000 C CNN
 F 1 "74LV595" H 8000 2500 50  0000 C CNN
 F 2 "Package_SO:TSSOP-16_4.4x5mm_P0.65mm" H 7750 1900 50  0001 C CNN
@@
 AR Path="/5A78E64E/5A7DC371/5A7A5871" Ref="U606"  Part="1"
 AR Path="/5A78E661/5A7DC371/5A7A5871" Ref="U806"  Part="1"
-F 0 "U606" H 9700 2600 50  0000 C CNN
+F 0 "U806" H 9700 2600 50  0000 C CNN
 F 1 "74LV595" H 9800 2500 50  0000 C CNN
 F 2 "Package_SO:TSSOP-16_4.4x5mm_P0.65mm" H 9550 1900 50  0001 C CNN
@@
 AR Path="/5A78E64E/5A7DC371/5A7ADAF8" Ref="U602"  Part="1"
 AR Path="/5A78E661/5A7DC371/5A7ADAF8" Ref="U802"  Part="1"
-F 0 "U602" H 2250 1575 50  0000 C CNN
+F 0 "U802" H 2250 1575 50  0000 C CNN
 F 1 "SN74LV86" H 2250 1484 50  0000 C CNN
 F 2 "Package_SO:TSSOP-14_4.4x5mm_P0.65mm" H 2250 1250 50  0001 C CNN
@@
 AR Path="/5A78E64E/5A7DC371/5A7B4C81" Ref="U604"  Part="1"
 AR Path="/5A78E661/5A7DC371/5A7B4C81" Ref="U804"  Part="1"
-F 0 "U604" H 4450 1667 50  0000 C CNN
+F 0 "U804" H 4450 1667 50  0000 C CNN
 F 1 "74LVC1G80" H 4450 1576 50  0000 C CNN
 F 2 "Package_TO_SOT_SMD:SOT-353_SC-70-5" H 4450 1350 50  0001 C CNN
@@
 AR Path="/5A78E64E/5A7DC371/5A7BEEBC" Ref="U601"  Part="1"
 AR Path="/5A78E661/5A7DC371/5A7BEEBC" Ref="U801"  Part="1"
-F 0 "U601" H 1800 4417 50  0000 C CNN
+F 0 "U801" H 1800 4417 50  0000 C CNN
 F 1 "74LVC3G14" H 1800 4326 50  0000 C CNN
 F 2 "Package_SO:VSSOP-8_2.3x2mm_P0.5mm" H 1800 4100 50  0001 C CNN
@@
 AR Path="/5A78E64E/5A7DC371/5A7C2776" Ref="U602"  Part="5"
 AR Path="/5A78E661/5A7DC371/5A7C2776" Ref="U802"  Part="5"
-F 0 "U602" H 6950 5900 50  0000 L CNN
+F 0 "U802" H 6950 5900 50  0000 L CNN
 F 1 "SN74LV86" H 6950 5800 50  0000 L CNN
 F 2 "Package_SO:TSSOP-14_4.4x5mm_P0.65mm" H 6800 5450 50  0001 C CNN
@@
 AR Path="/5A78E64E/5A7DC371/5A7C605D" Ref="U604"  Part="2"
 AR Path="/5A78E661/5A7DC371/5A7C605D" Ref="U804"  Part="2"
-F 0 "U604" H 8450 5800 50  0000 L CNN
+F 0 "U804" H 8450 5800 50  0000 L CNN
 F 1 "74LVC1G80" H 8450 5700 50  0000 L CNN
 F 2 "Package_TO_SOT_SMD:SOT-353_SC-70-5" H 8400 5400 50  0001 C CNN
@@
 AR Path="/5A78E64E/5A7DC371/5A81E8DA" Ref="C607"  Part="1"
 AR Path="/5A78E661/5A7DC371/5A81E8DA" Ref="C807"  Part="1"
-F 0 "C607" H 2515 4346 50  0000 L CNN
+F 0 "C807" H 2515 4346 50  0000 L CNN
 F 1 "DNP" H 2515 4255 50  0000 L CNN
 F 2 "Capacitor_SMD:C_0603_1608Metric" H 2438 4150 50  0001 C CNN
@@
 AR Path="/5A78E64E/5A7DC371/5A82356F" Ref="C601"  Part="1"
 AR Path="/5A78E661/5A7DC371/5A82356F" Ref="C801"  Part="1"
-F 0 "C601" H 6265 5496 50  0000 L CNN
+F 0 "C801" H 6265 5496 50  0000 L CNN
 F 1 "0u1F" H 6265 5405 50  0000 L CNN
 F 2 "Capacitor_SMD:C_0603_1608Metric" H 6188 5300 50  0001 C CNN
@@
 AR Path="/5A78E64E/5A7DC371/5A823695" Ref="C604"  Part="1"
 AR Path="/5A78E661/5A7DC371/5A823695" Ref="C804"  Part="1"
-F 0 "C604" H 9065 5496 50  0000 L CNN
+F 0 "C804" H 9065 5496 50  0000 L CNN
 F 1 "0u1F" H 9065 5405 50  0000 L CNN
 F 2 "Capacitor_SMD:C_0603_1608Metric" H 8988 5300 50  0001 C CNN
@@
 AR Path="/5A78E64E/5A7DC371/5A823707" Ref="C603"  Part="1"
 AR Path="/5A78E661/5A7DC371/5A823707" Ref="C803"  Part="1"
-F 0 "C603" H 7915 5496 50  0000 L CNN
+F 0 "C803" H 7915 5496 50  0000 L CNN
 F 1 "0u1F" H 7915 5405 50  0000 L CNN
 F 2 "Capacitor_SMD:C_0603_1608Metric" H 7838 5300 50  0001 C CNN
@@
 AR Path="/5A78E64E/5A7DC371/5A823767" Ref="C606"  Part="1"
 AR Path="/5A78E661/5A7DC371/5A823767" Ref="C806"  Part="1"
-F 0 "C606" H 9865 5496 50  0000 L CNN
+F 0 "C806" H 9865 5496 50  0000 L CNN
 F 1 "0u1F" H 9865 5405 50  0000 L CNN
 F 2 "Capacitor_SMD:C_0603_1608Metric" H 9788 5300 50  0001 C CNN
@@
 AR Path="/5A78E64E/5A7DC371/5A8237CD" Ref="C605"  Part="1"
 AR Path="/5A78E661/5A7DC371/5A8237CD" Ref="C805"  Part="1"
-F 0 "C605" H 9615 5496 50  0000 L CNN
+F 0 "C805" H 9615 5496 50  0000 L CNN
 F 1 "0u1F" H 9615 5405 50  0000 L CNN
 F 2 "Capacitor_SMD:C_0603_1608Metric" H 9538 5300 50  0001 C CNN
@@
 $Comp
 L CommsCard:74LVC3G14 U601
-U 3 1 5A86AE5A
+U 2 1 5A86AE5A
 P 3050 4100
 AR Path="/5A78E64E/5A7DC371/5A86AE5A" Ref="U601"  Part="3"
@@
 F 3 "http://www.ti.com/lit/ds/symlink/sn74lvc3g14.pdf" H 3050 4100 50  0001 C CNN
 F 4 "SN74LVC3G14DCUR" H 3050 4100 50  0001 C CNN "mpn"
-	3    3050 4100
+	2    3050 4100
 	1    0    0    -1
 $EndComp
@@
 AR Path="/5A78E64E/5A7DC371/5A86AF6E" Ref="U601"  Part="4"
 AR Path="/5A78E661/5A7DC371/5A86AF6E" Ref="U801"  Part="4"
-F 0 "U601" H 5750 5900 50  0000 C CNN
+F 0 "U801" H 5750 5900 50  0000 C CNN
 F 1 "74LVC3G14" H 5800 5800 50  0000 C CNN
 F 2 "Package_SO:VSSOP-8_2.3x2mm_P0.5mm" H 5550 5450 50  0001 C CNN
@@
 AR Path="/5A78E64E/5A7DC371/5A877722" Ref="U603"  Part="1"
 AR Path="/5A78E661/5A7DC371/5A877722" Ref="U803"  Part="1"
-F 0 "U603" H 3100 2515 50  0000 C CNN
+F 0 "U803" H 3100 2515 50  0000 C CNN
 F 1 "501BMILF" H 3100 2424 50  0000 C CNN
 F 2 "Package_SO:SOIC-8_3.9x4.9mm_P1.27mm" H 3100 2050 50  0001 C CNN
@@
 AR Path="/5A78E64E/5A7DC371/5A89CAC8" Ref="C602"  Part="1"
 AR Path="/5A78E661/5A7DC371/5A89CAC8" Ref="C802"  Part="1"
-F 0 "C602" H 7465 5496 50  0000 L CNN
+F 0 "C802" H 7465 5496 50  0000 L CNN
 F 1 "0u1F" H 7465 5405 50  0000 L CNN
 F 2 "Capacitor_SMD:C_0603_1608Metric" H 7388 5300 50  0001 C CNN
@@
 AR Path="/5A78E64E/5A7DC371/5A8A39CD" Ref="U602"  Part="2"
 AR Path="/5A78E661/5A7DC371/5A8A39CD" Ref="U802"  Part="2"
-F 0 "U602" H 6700 1825 50  0000 C CNN
+F 0 "U802" H 6700 1825 50  0000 C CNN
 F 1 "SN74LV86" H 6700 1734 50  0000 C CNN
 F 2 "Package_SO:TSSOP-14_4.4x5mm_P0.65mm" H 6700 1500 50  0001 C CNN
@@
 AR Path="/5A78E64E/5A7DC371/5A8B4217" Ref="U602"  Part="3"
 AR Path="/5A78E661/5A7DC371/5A8B4217" Ref="U802"  Part="3"
-F 0 "U602" H 10400 2275 50  0000 C CNN
+F 0 "U802" H 10400 2275 50  0000 C CNN
 F 1 "SN74LV86" H 10400 2184 50  0000 C CNN
 F 2 "Package_SO:TSSOP-14_4.4x5mm_P0.65mm" H 10400 1950 50  0001 C CNN
@@
 Connection ~ 9500 4850
 Connection ~ 9500 6000
+Text Label 3700 1900 0    50   ~ 0
+2xCLOCK
+Text Label 2750 1250 0    50   ~ 0
+RAW_BIPHASE
 $EndSCHEMATC
