File: design/LOSComms.sch (KiCad schematic (older format))
At the start: 13 parts, among them U601 74LVC3G14, U602 SN74LV86, U603 501BMILF, U604 74LVC1G80, U605 74LV595, U606 74LV595

Commit message: Adding more LOS detail
Parts:
- removed C607: DNP, Capacitor_SMD:C_0603_1608Metric, symbol Device:C
- U601: value 74LVC3G14 -> 74LVC14; footprint Package_SO:VSSOP-8_2.3x2mm_P0.5mm -> Package_SO:TSSOP-14_4.4x5mm_P0.65mm; mpn SN74LVC3G14DCUR -> 74LVC14AT14-13
Connections:
- wire segments 83 -> 80

Commit message: Changing to dual-gate inverters for delay line
Parts:
- removed unit 4 of U601
- added C607: DNP, Capacitor_SMD:C_0603_1608Metric, symbol Device:C
- added unit 3 of U601
- U601: value 74LVC14 -> 74LVC3G14; footprint Package_SO:TSSOP-14_4.4x5mm_P0.65mm -> Package_TO_SOT_SMD:SOT-363_SC-70-6; symbol CommsCard:74LVC3G14 -> CommsCard:74LVC2G14
Connections:
- wire segments 80 -> 83

Commit message: Finalizing FC1 --- ish
Connections:
- net CLK: now also U602.13; no longer U602.2
- net DATA: now also U602.12; no longer U602.1
- net RAW_BIPHASE: now also U602.11; no longer U602.3
Changed lines of the file:
@@
 $Comp
 L Logic_74xx:74LS86 U602
-U 1 1 5A7ADAF8
+U 4 1 5A7ADAF8
 P 2250 1250
 AR Path="/5A78E64E/5A7DC371/5A7ADAF8" Ref="U602"  Part="1"
-AR Path="/5A78E661/5A7DC371/5A7ADAF8" Ref="U802"  Part="1"
+AR Path="/5A78E661/5A7DC371/5A7ADAF8" Ref="U802"  Part="4"
 F 0 "U802" H 2250 1575 50  0000 C CNN
 F 1 "SN74LV86" H 2250 1484 50  0000 C CNN
@@
 F 3 "http://www.ti.com/lit/ds/symlink/sn74lv86a-ep.pdf" H 2250 1250 50  0001 C CNN
 F 4 "SN74LV86ATPWREP" H 2250 1250 50  0001 C CNN "mpn"
-	1    2250 1250
+	4    2250 1250
 	1    0    0    -1
 $EndComp
