File: design/power.sch (KiCad schematic (older format))
At the start: 0 parts

Commit message: Adding LT39509 regulator for voltage levels
Parts:
- added C?: 2u2F, Capacitor_SMD:C_0805_2012Metric, symbol Device:C_Small
- added C? (x4): 0u1F, Capacitor_SMD:C_0603_1608Metric, symbol Device:C_Small
- added C? (x2): 10uF, Capacitor_SMD:C_0805_2012Metric, symbol Device:C_Small
- added C? (x2): 22nF, Capacitor_SMD:C_0603_1608Metric, symbol Device:C_Small
- added D? (x2): MBRM140, Diode_SMD:D_Powermite2_AK, symbol Device:D_Schottky_Small_ALT
- added J?: Conn_01x02, Connector_Phoenix_MC:PhoenixContact_MC_1,5_2-G-5.08_1x02_P5.08mm_Horizontal, symbol Connector_Generic:Conn_01x02
- added L?: 4u7H, Inductor_SMD:L_Abracon_ASPI-3012S, symbol Device:L
- added L?: 6u8H, Inductor_SMD:L_Abracon_ASPI-3012S, symbol Device:L
- added R?: 16k9, Resistor_SMD:R_0603_1608Metric, symbol Device:R
- added R? (x2): 10k, Resistors_SMD:R_0603, symbol Device:R
- added R?: 31k6, Resistors_SMD:R_0603, symbol Device:R
- added R?: 52k3, Resistors_SMD:R_0603, symbol Device:R
- added U? (x3): LT3509EMSE, symbol CommsCard:LT3509EMSE
Connections:
- net labels added: +3.3V, +5V, GND
- wire segments 0 -> 61

Commit message: Finished ERC
Parts:
- gave numbers to parts that had none: 20
Connections:
- net labels added: PWR_IN
- wire segments 61 -> 63

Commit message: Swapping FT4232 for VQFN and finalizing mpns
Parts:
- U201: footprint (none) -> Package_SO:MSOP-16-1EP_3x4mm_P0.5mm_EP1.65x2.85mm_ThermalVias; mpn (none) -> LT3509EMSE#PBF
Changed lines of the file:
@@
-$Comp
-L CommsCard:LT3509EMSE U201
-U 1 1 5A7E3A66
-P 5600 2500
-F 0 "U201" H 5600 2975 50  0000 C CNN
-F 1 "LT3509EMSE" H 5600 2884 50  0000 C CNN
-F 2 "" H 5600 2400 50  0001 C CNN
-F 3 "" H 5600 2400 50  0001 C CNN
-	1    5600 2500
-	1    0    0    -1
-$EndComp
-$Comp
-L CommsCard:LT3509EMSE U201
-U 2 1 5A7E3AD8
-P 5600 3900
-F 0 "U201" H 5600 4375 50  0000 C CNN
-F 1 "LT3509EMSE" H 5600 4284 50  0000 C CNN
-F 2 "" H 5600 3800 50  0001 C CNN
-F 3 "" H 5600 3800 50  0001 C CNN
-F 4 "~" H 5600 3900 50  0001 C CNN "mpn"
-	2    5600 3900
-	1    0    0    -1
-$EndComp
 $Comp
 L CommsCard:LT3509EMSE U201
@@
 F 0 "U201" H 4050 4028 50  0000 C CNN
 F 1 "LT3509EMSE" H 4050 3937 50  0000 C CNN
-F 2 "" H 4050 3150 50  0001 C CNN
-F 3 "" H 4050 3150 50  0001 C CNN
-F 4 "~" H 4050 3250 50  0001 C CNN "mpn"
+F 2 "Package_SO:MSOP-16-1EP_3x4mm_P0.5mm_EP1.65x2.85mm_ThermalVias" H 4050 3150 50  0001 C CNN
+F 3 "http://www.linear.com/docs/27202" H 4050 3150 50  0001 C CNN
+F 4 "LT3509EMSE#PBF" H 4050 3250 50  0001 C CNN "mpn"
 	3    4050 3250
 	1    0    0    -1
@@
 	1    0    0    -1
 $EndComp
-Connection ~ 6050 2400
 Wire Wire Line
 	5950 2250 5950 2200
@@
 Wire Wire Line
 	6900 4150 6800 4150
+$Comp
+L CommsCard:LT3509EMSE U201
+U 1 1 5A85BAAB
+P 5600 2500
+F 0 "U201" H 5600 3278 50  0000 C CNN
+F 1 "LT3509EMSE" H 5600 3187 50  0000 C CNN
+F 2 "Package_SO:MSOP-16-1EP_3x4mm_P0.5mm_EP1.65x2.85mm_ThermalVias" H 5600 2400 50  0001 C CNN
+F 3 "http://www.linear.com/docs/27202" H 5600 2400 50  0001 C CNN
+F 4 "LT3509EMSE#PBF" H 5600 2500 50  0001 C CNN "mpn"
+	1    5600 2500
+	1    0    0    -1
+$EndComp
+$Comp
+L CommsCard:LT3509EMSE U201
+U 2 1 5A85BB2F
+P 5600 3900
+F 0 "U201" H 5600 4678 50  0000 C CNN
+F 1 "LT3509EMSE" H 5600 4587 50  0000 C CNN
+F 2 "Package_SO:MSOP-16-1EP_3x4mm_P0.5mm_EP1.65x2.85mm_ThermalVias" H 5600 3800 50  0001 C CNN
+F 3 "http://www.linear.com/docs/27202" H 5600 3800 50  0001 C CNN
+F 4 "LT3509EMSE#PBF" H 5600 3900 50  0001 C CNN "mpn"
+	2    5600 3900
+	1    0    0    -1
+$EndComp
+Connection ~ 6050 2400
 $EndSCHEMATC

Commit message: Updating schematic for layout
Parts:
- C202, C203, C206, C207: mpn UMJ107BB7104KAHT -> CL10B104KO8WPNC
- R202, R203, R204, R205: footprint Resistors_SMD:R_0603 -> Resistor_SMD:R_0603_1608Metric
Changed lines of the file:
@@
 F 1 "0u1F" H 3292 2655 50  0000 L CNN
 F 2 "Capacitor_SMD:C_0603_1608Metric" H 3200 2700 50  0001 C CNN
-F 3 "https://www.yuden.co.jp/productdata/catalog/mlcc_all_e.pdf" H 3200 2700 50  0001 C CNN
-F 4 "UMJ107BB7104KAHT" H 3200 2700 50  0001 C CNN "mpn"
+F 3 "http://www.samsungsem.com/kr/support/product-search/mlcc/CL10B104KO8WPNC.jsp" H 3200 2700 50  0001 C CNN
+F 4 "CL10B104KO8WPNC" H 3200 2700 50  0001 C CNN "mpn"
 	1    3200 2700
 	1    0    0    -1
@@
 F 1 "0u1F" H 3642 2655 50  0000 L CNN
 F 2 "Capacitor_SMD:C_0603_1608Metric" H 3550 2700 50  0001 C CNN
-F 3 "https://www.yuden.co.jp/productdata/catalog/mlcc_all_e.pdf" H 3550 2700 50  0001 C CNN
-F 4 "UMJ107BB7104KAHT" H 3550 2700 50  0001 C CNN "mpn"
+F 3 "http://www.samsungsem.com/kr/support/product-search/mlcc/CL10B104KO8WPNC.jsp" H 3550 2700 50  0001 C CNN
+F 4 "CL10B104KO8WPNC" H 3550 2700 50  0001 C CNN "mpn"
 	1    3550 2700
 	1    0    0    -1
@@
 F 0 "R203" H 6180 4304 50  0000 R CNN
 F 1 "10k" H 6180 4395 50  0000 R CNN
-F 2 "Resistors_SMD:R_0603" V 6180 4350 50  0001 C CNN
+F 2 "Resistor_SMD:R_0603_1608Metric" V 6180 4350 50  0001 C CNN
 F 3 "http://www.te.com/commerce/DocumentDelivery/DDEController?Action=srchrtrv&DocNm=1773204&DocType=DS&DocLang=English" H 6250 4350 50  0001 C CNN
 F 4 "CRG0603J10K" H 6250 4350 50  0001 C CNN "mpn"
@@
 F 0 "R204" H 6580 2704 50  0000 R CNN
 F 1 "31k6" H 6580 2795 50  0000 R CNN
-F 2 "Resistors_SMD:R_0603" V 6580 2750 50  0001 C CNN
+F 2 "Resistor_SMD:R_0603_1608Metric" V 6580 2750 50  0001 C CNN
 F 3 "http://www.vishay.com/docs/20035/dcrcwe3.pdf" H 6650 2750 50  0001 C CNN
 F 4 "CRCW060331K6FKEA" H 6650 2750 50  0001 C CNN "mpn"
@@
 F 0 "R205" H 6580 4104 50  0000 R CNN
 F 1 "52k3" H 6580 4195 50  0000 R CNN
-F 2 "Resistors_SMD:R_0603" V 6580 4150 50  0001 C CNN
+F 2 "Resistor_SMD:R_0603_1608Metric" V 6580 4150 50  0001 C CNN
 F 3 "http://www.vishay.com/docs/20035/dcrcwe3.pdf" H 6650 4150 50  0001 C CNN
 F 4 "CRCW060352K3FKEA" H 6650 4150 50  0001 C CNN "mpn"
@@
 F 0 "R202" H 6180 2954 50  0000 R CNN
 F 1 "10k" H 6180 3045 50  0000 R CNN
-F 2 "Resistors_SMD:R_0603" V 6180 3000 50  0001 C CNN
+F 2 "Resistor_SMD:R_0603_1608Metric" V 6180 3000 50  0001 C CNN
 F 3 "http://www.te.com/commerce/DocumentDelivery/DDEController?Action=srchrtrv&DocNm=1773204&DocType=DS&DocLang=English" H 6250 3000 50  0001 C CNN
 F 4 "CRG0603J10K" H 6250 3000 50  0001 C CNN "mpn"
@@
 F 1 "0u1F" H 6142 2255 50  0000 L CNN
 F 2 "Capacitor_SMD:C_0603_1608Metric" H 6050 2300 50  0001 C CNN
-F 3 "https://www.yuden.co.jp/productdata/catalog/mlcc_all_e.pdf" H 6050 2300 50  0001 C CNN
-F 4 "UMJ107BB7104KAHT" H 6050 2300 50  0001 C CNN "mpn"
+F 3 "http://www.samsungsem.com/kr/support/product-search/mlcc/CL10B104KO8WPNC.jsp" H 6050 2300 50  0001 C CNN
+F 4 "CL10B104KO8WPNC" H 6050 2300 50  0001 C CNN "mpn"
 	1    6050 2300
 	1    0    0    -1
@@
 F 1 "0u1F" H 6142 3655 50  0000 L CNN
 F 2 "Capacitor_SMD:C_0603_1608Metric" H 6050 3700 50  0001 C CNN
-F 3 "https://www.yuden.co.jp/productdata/catalog/mlcc_all_e.pdf" H 6050 3700 50  0001 C CNN
-F 4 "UMJ107BB7104KAHT" H 6050 3700 50  0001 C CNN "mpn"
+F 3 "http://www.samsungsem.com/kr/support/product-search/mlcc/CL10B104KO8WPNC.jsp" H 6050 3700 50  0001 C CNN
+F 4 "CL10B104KO8WPNC" H 6050 3700 50  0001 C CNN "mpn"
 	1    6050 3700
 	1    0    0    -1

Commit message: Label power nets
Connections:
- net labels added: BOOST1, BOOST2, DA1, DA2, FB1, FB2, SW1, SW2
Changed lines of the file:
@@
 $EndComp
 Connection ~ 6050 2400
+Text Label 6000 2600 1    50   ~ 0
+DA1
+Text Label 6000 4000 1    50   ~ 0
+DA2
+Text Label 6000 4150 0    50   ~ 0
+FB2
+Text Label 6000 2750 0    50   ~ 0
+FB1
+Text Label 5950 3600 0    50   ~ 0
+BOOST2
+Text Label 5950 2200 0    50   ~ 0
+BOOST1
+Text Label 6350 2400 0    20   ~ 0
+SW1
+Text Label 6350 3800 0    20   ~ 0
+SW2
 $EndSCHEMATC
