File: design/USB.sch (KiCad schematic (older format))
At the start: 10 parts, among them J901 USB_B, U901 ADUM3160

Commit message: Adding more LOS detail
Changed lines of the file:
@@
 AR Path="/5A8C396A/5A8C44FE" Ref="U901"  Part="1"
 AR Path="/5A8D14B5/5A8C44FE" Ref="U1001"  Part="1"
-F 0 "U901" H 5200 4028 50  0000 C CNN
+F 0 "U1001" H 5200 4028 50  0000 C CNN
 F 1 "ADUM3160" H 5200 3937 50  0000 C CNN
 F 2 "Package_SO:SOIC-16W_7.5x10.3mm_P1.27mm" H 5200 2550 50  0001 C CNN
@@
 AR Path="/5A8C396A/5A8C4970" Ref="J901"  Part="1"
 AR Path="/5A8D14B5/5A8C4970" Ref="J1001"  Part="1"
-F 0 "J901" H 2655 3526 50  0000 C CNN
+F 0 "J1001" H 2655 3526 50  0000 C CNN
 F 1 "USB_B" H 2655 3526 50  0001 C CNN
 F 2 "Connector_USB:USB_Micro-B_Amphenol_10103594-0001LF_Horizontal" H 2750 3100 50  0001 C CNN
@@
 AR Path="/5A8C396A/5A8C4F26" Ref="R902"  Part="1"
 AR Path="/5A8D14B5/5A8C4F26" Ref="R1002"  Part="1"
-F 0 "R902" V 4250 3250 50  0000 C CNN
+F 0 "R1002" V 4250 3250 50  0000 C CNN
 F 1 "24R" V 4150 3250 50  0000 C CNN
 F 2 "Resistor_SMD:R_0402_1005Metric" H 4050 3250 50  0001 C CNN
@@
 AR Path="/5A8C396A/5A8C58B8" Ref="C901"  Part="1"
 AR Path="/5A8D14B5/5A8C58B8" Ref="C1001"  Part="1"
-F 0 "C901" H 3515 3746 50  0000 L CNN
+F 0 "C1001" H 3515 3746 50  0000 L CNN
 F 1 "0u1F" H 3515 3655 50  0000 L CNN
 F 2 "Capacitor_SMD:C_0603_1608Metric" H 3438 3550 50  0001 C CNN
@@
 AR Path="/5A8C396A/5A8C58F7" Ref="C902"  Part="1"
 AR Path="/5A8D14B5/5A8C58F7" Ref="C1002"  Part="1"
-F 0 "C902" H 4565 3746 50  0000 L CNN
+F 0 "C1002" H 4565 3746 50  0000 L CNN
 F 1 "0u1F" H 4565 3655 50  0000 L CNN
 F 2 "Capacitor_SMD:C_0603_1608Metric" H 4488 3550 50  0001 C CNN
@@
 AR Path="/5A8C396A/5A8C93E9" Ref="R903"  Part="1"
 AR Path="/5A8D14B5/5A8C93E9" Ref="R1003"  Part="1"
-F 0 "R903" V 5804 3150 50  0000 C CNN
+F 0 "R1003" V 5804 3150 50  0000 C CNN
 F 1 "24R" V 5895 3150 50  0000 C CNN
 F 2 "Resistor_SMD:R_0402_1005Metric" H 6000 3150 50  0001 C CNN
@@
 AR Path="/5A8C396A/5A8C5368" Ref="R901"  Part="1"
 AR Path="/5A8D14B5/5A8C5368" Ref="R1001"  Part="1"
-F 0 "R901" V 3854 3150 50  0000 C CNN
+F 0 "R1001" V 3854 3150 50  0000 C CNN
 F 1 "24R" V 3945 3150 50  0000 C CNN
 F 2 "Resistor_SMD:R_0402_1005Metric" H 4050 3150 50  0001 C CNN
@@
 AR Path="/5A8C396A/5A8CAB7B" Ref="R904"  Part="1"
 AR Path="/5A8D14B5/5A8CAB7B" Ref="R1004"  Part="1"
-F 0 "R904" V 6200 3250 50  0000 C CNN
+F 0 "R1004" V 6200 3250 50  0000 C CNN
 F 1 "24R" V 6100 3250 50  0000 C CNN
 F 2 "Resistor_SMD:R_0402_1005Metric" H 6000 3250 50  0001 C CNN
@@
 L Device:C_Small C904
 U 1 1 5A8CE0CB
-P 6300 2700
+P 5800 3900
 AR Path="/5A8C396A/5A8CE0CB" Ref="C904"  Part="1"
 AR Path="/5A8D14B5/5A8CE0CB" Ref="C1004"  Part="1"
-F 0 "C904" H 6415 2746 50  0000 L CNN
+F 0 "C1004" H 5915 3946 50  0000 L CNN
+F 1 "0u1F" H 5915 3855 50  0000 L CNN
+F 2 "Capacitor_SMD:C_0603_1608Metric" H 5838 3750 50  0001 C CNN
+F 3 "http://www.samsungsem.com/kr/support/product-search/mlcc/CL10B104KO8WPNC.jsp" H 5800 3900 50  0001 C CNN
+F 4 "CL10B104KO8WPNC" H 5800 3900 50  0001 C CNN "mpn"
+	1    5800 3900
+	1    0    0    -1
+$EndComp
+$Comp
+L Device:C_Small C903
+U 1 1 5A8CE121
+P 6300 2700
+AR Path="/5A8C396A/5A8CE121" Ref="C903"  Part="1"
+AR Path="/5A8D14B5/5A8CE121" Ref="C1003"  Part="1"
+F 0 "C1003" H 6415 2746 50  0000 L CNN
 F 1 "0u1F" H 6415 2655 50  0000 L CNN
 F 2 "Capacitor_SMD:C_0603_1608Metric" H 6338 2550 50  0001 C CNN
@@
 	1    0    0    -1
 $EndComp
-$Comp
-L Device:C_Small C903
-U 1 1 5A8CE121
-P 5800 3900
-AR Path="/5A8C396A/5A8CE121" Ref="C903"  Part="1"
-AR Path="/5A8D14B5/5A8CE121" Ref="C1003"  Part="1"
-F 0 "C903" H 5915 3946 50  0000 L CNN
-F 1 "0u1F" H 5915 3855 50  0000 L CNN
-F 2 "Capacitor_SMD:C_0603_1608Metric" H 5838 3750 50  0001 C CNN
-F 3 "http://www.samsungsem.com/kr/support/product-search/mlcc/CL10B104KO8WPNC.jsp" H 5800 3900 50  0001 C CNN
-F 4 "CL10B104KO8WPNC" H 5800 3900 50  0001 C CNN "mpn"
-	1    5800 3900
-	1    0    0    -1
-$EndComp
